File: _autosave-afx-01.kicad_pcb (KiCad board)
At the start: 2 copper layers, 91.4 x 116.8 mm, 114 parts, among them J1 HeadphoneOut, J2 MicIn, P1 CONN_02X05, P2 CONN_02X05, U1 ADA_SSD1306_I2C, U2 Teensy_3.1, U3 SAM2695, U4 MicroSD_Adapter, U5 SSD1306, X1 12MHz

Commit message: Moving on to proto6!
Parts:
- removed U5: SSD1306, afx-01:SSD1306_XL
- moved C11 119.3 mm to (85.6, 150.9)
- moved C12 119.3 mm to (98.3, 154.2)
- moved C20 119.3 mm to (80.0, 151.1)
- moved J1 119.3 mm to (92.1, 142.9)
- moved J2 119.3 mm to (68.6, 156.8)
- moved P1 119.3 mm to (112.4, 184.8)
- moved P2 119.3 mm to (122.6, 184.8)
- moved R18 119.3 mm to (99.1, 188.6)
- moved R19 119.3 mm to (92.7, 188.6)
- moved R4 119.3 mm to (84.1, 146.3)
- moved R5 119.3 mm to (98.3, 151.1)
- moved R7 119.3 mm to (80.0, 144.8)
- moved REF** 119.3 mm to (70.5, 144.8)
- moved U1 119.3 mm to (113.0, 144.8)
- moved U4 119.3 mm to (116.2, 165.1)
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Routing:
- net GND: track 941.3 -> 608.6 mm, vias 14 -> 7
- net VCC: track 748.1 -> 549.5 mm, vias 18 -> 12
- net /SwitchMatrix/SDA: track 151.7 -> 0.45 mm, vias 4 -> 0
- net /SwitchMatrix/SCL: track 149.8 -> 0.00 mm, vias 2 -> 0
- net Net-(MCP2-Pad23): track 133.0 -> 6.60 mm, vias 1 -> 0
- net Net-(MCP2-Pad27): track 126.5 -> 6.60 mm, vias 1 -> 0
- net AGND: track 196.6 -> 93.3 mm
- net Net-(ENC1-Pad4): track 93.8 -> 0.00 mm, vias 1 -> 0
- net /SoundBoard/MIDIIN: track 93.2 -> 3.30 mm
- net Net-(MCP1-Pad19): track 94.5 -> 6.60 mm, vias 2 -> 0
- net /SwitchMatrix/ENCB: track 88.0 -> 2.71 mm
- net Net-(MCP1-Pad17): track 91.3 -> 6.60 mm, vias 2 -> 0
- net /SwitchMatrix/ENCA: track 84.7 -> 2.71 mm
- net Net-(C20-Pad1): track 82.0 -> 0.00 mm, vias 2 -> 0
- net Net-(C11-Pad1): track 77.7 -> 0.00 mm, vias 2 -> 0
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Other:
- board size 91.4 x 116.8 mm -> 114.3 x 110.5 mm
