File: _autosave-afx-01.kicad_pcb (KiCad board)
At the start: 2 copper layers, 116.2 x 110.5 mm, 198 parts, among them J1 HeadphoneOut, J10 Mono_AudioConnector, J11 Mono_AudioConnector, J12 Mono_AudioConnector, J13 Mono_AudioConnector, J14 Mono_AudioConnector, J15 Mono_AudioConnector, J16 Mono_AudioConnector, J17 Mono_AudioConnector, J18 Mono_AudioConnector, J2 MicIn, J3 Mono_AudioConnector, J4 Mono_AudioConnector, J5 Mono_AudioConnector, J6 Mono_AudioConnector, J7 Mono_AudioConnector, J8 Mono_AudioConnector, J9 Mono_AudioConnector, P1 CONN_02X05, P2 CONN_02X05, Q1 Q_NPN_BCE, Q2 Q_NPN_BCE, Q3 Q_NPN_BCE, Q4 Q_NPN_BCE, U1 ADA_SSD1306_I2C, U13 MCP6004, U2 Teensy_3.1, U3 SAM2695, U4 MicroSD_Adapter, U5 MCP1703, U6 OPA4171, U7 OPA4171, U8 AD5676, X1 12MHz

Commit message: UPDATEUPDATES!!!
Parts:
- added JP3: JUMPER3, Zetaohm:Jumper_3way, F.Cu at (88.6, 143.4)
- added Q5, Q6: BSS138, Housings_SOT-23_SOT-143_TSOT-6:SOT-23, F.Cu at (88.6, 143.4)
- added R72, R73: 4.7k, Resistors_SMD:R_0805_HandSoldering, F.Cu at (88.6, 143.4)
- P2: value CONN_02X05 -> CONN_02X08; footprint ab2_header:AB2_HDR_M05-2V -> Pin_Headers:Pin_Header_Angled_2x08; moved to F.Cu
- U2: footprint Zetaohm:Teensy3.1 -> Zetaohm:Teensy3.1_Min_I2C2
- moved J2 230.2 mm to (308.0, 73.5)
- moved U8 152.8 mm to (40.6, 80.0)
- moved Q1 133.3 mm to (158.4, 114.1)
- moved J15 130.7 mm to (205.3, 84.5)
- moved J16 124.3 mm to (205.3, 100.6)
- moved Q3 124.2 mm to (178.7, 112.9)
- moved P2 119.6 mm to (88.6, 143.4), turned to 0 degrees
- moved J1 117.9 mm to (288.7, 73.5)
- moved R62 116.8 mm to (201.6, 117.4)
- moved J13 116.0 mm to (188.6, 84.5)
- moved Q4 115.6 mm to (151.4, 114.1)
- moved R54 112.6 mm to (185.8, 117.4)
- moved C40 111.1 mm to (191.0, 111.1)
- moved C37 109.4 mm to (206.7, 119.7)
- moved J14 108.8 mm to (188.6, 100.6)
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Connections:
- MCP1 pad 8: SCL0 -> SCL0_5v
- MCP1 pad 9: SDA0 -> SDA0_5v
- MCP2 pad 8: SCL0 -> SCL0_5v
- MCP2 pad 9: SDA0 -> SDA0_5v
- U5 pad 2: +5V -> Net-(JP3-Pad1)

Commit message: Added Touch Capacitive Panel
Parts:
- removed C20: 1µfT, Capacitors_SMD:C_0805_HandSoldering
- removed C21: 220pF, Capacitors_SMD:C_0805_HandSoldering
- removed J1: HeadphoneOut, Zetaohm:Switchcraft_3.5mm_SMD_Stereo
- removed J2: MicIn, Zetaohm:Switchcraft_3.5mm_SMD_Stereo
- removed the J3 at (27.9, 162.6)
- removed the J5 at (44.5, 161.3)
- removed the J7 at (59.7, 159.9)
- removed the J9 at (72.4, 160.0)
- removed R7: 4.7k, Resistors_SMD:R_0805_HandSoldering
- added G***: CAPACITIVE_FACEPLATE, Zetaohm:FACEPLATEV1, F.Cu at (213.3, 91.2)
- added J11: Mono_AudioConnector, Zetaohm:THONKICONN, F.Cu at (24.8, 139.3)
- added J15: Mono_AudioConnector, Zetaohm:THONKICONN, F.Cu at (44.9, 127.6)
- added J16: Mono_AudioConnector, Zetaohm:THONKICONN, F.Cu at (54.4, 127.6)
- added J17: Mono_AudioConnector, Zetaohm:THONKICONN, F.Cu at (43.6, 139.3)
- added J19: Mono_AudioConnector, Zetaohm:THONKICONN, F.Cu at (82.7, 127.6)
- added J20: Mono_AudioConnector, Zetaohm:THONKICONN, F.Cu at (81.2, 139.3)
- added J21: Mono_AudioConnector, Zetaohm:THONKICONN, F.Cu at (120.4, 127.6)
- added J21: Mono_AudioConnector, Zetaohm:THONKICONN, F.Cu at (111.0, 127.6)
- added J22: Mono_AudioConnector, Zetaohm:THONKICONN, F.Cu at (109.5, 139.3)
- added LED17: WS2812b, Zetaohm:WS2812b_SMD, F.Cu at (54.8, 114.5)
- added LED18: WS2812b, Zetaohm:WS2812b_SMD, F.Cu at (72.2, 114.5)
- added LED19: WS2812b, Zetaohm:WS2812b_SMD, F.Cu at (89.6, 114.5)
- added LED20: WS2812b, Zetaohm:WS2812b_SMD, F.Cu at (107.0, 114.5)
- added R74: 1k, Resistors_SMD:R_0603_HandSoldering, F.Cu at (56.5, 191.9)
- added R75: 1k, Resistors_SMD:R_0603_HandSoldering, F.Cu at (52.1, 191.9)
- added R76: 1k, Resistors_SMD:R_0603_HandSoldering, F.Cu at (56.5, 186.0)
- added R77: 1k, Resistors_SMD:R_0603_HandSoldering, F.Cu at (52.1, 186.0)
- added U10: MicroSD_Connector, Zetaohm:AMPHENOL_MICROSD, F.Cu at (104.2, 11.4)
- added U9: 3_pin_stereo, Zetaohm:KOBICONN_ST, F.Cu at (118.6, 139.3)
- C1, C2, C3, C4: value 100µf -> 100uf; footprint Capacitors_SMD:C_0805_HandSoldering -> Capacitors_SMD:C_0603_HandSoldering
- C10, C11, C12, C13, C14, C15, C16, C17, C18, C19, C22, C23, C24, C25, C26, C27, C28, C29, C30, C31, C32, C33, C34, C35, C36, C37, C38, C39, C40, C5, C6, C7, C8, C9, L1: footprint Capacitors_SMD:C_0805_HandSoldering -> Capacitors_SMD:C_0603_HandSoldering
- MIDI_IN1, MIDI_OUT1: moved to F.Cu
- P2: footprint Pin_Headers:Pin_Header_Angled_2x08 -> Pin_Headers:Pin_Header_Straight_2x08
- Q1, Q2, Q3, Q4: value Q_NPN_BCE -> BSS138
- R1, R10, R11, R12, R13, R14, R15, R16, R17, R18, R19, R2, R20, R21, R22, R23, R24, R25, R26, R27, R28, R29, R3, R30, R31, R32, R33, R34, R35, R36, R37, R38, R39, R4, R40, R41, R42, R43, R44, R45, R46, R47, R48, R49, R5, R50, R51, R52, R53, R54, R55, R56, R57, R58, R59, R6, R60, R61, R62, R63, R64, R65, R66, R67, R68, R69, R70, R71, R72, R73, R8, R9: footprint Resistors_SMD:R_0805_HandSoldering -> Resistors_SMD:R_0603_HandSoldering
- moved JP1 245.5 mm to (52.1, 20.3)
- moved JP2 237.0 mm to (48.5, 16.2)
- moved C35 235.5 mm to (47.6, 186.0)
- moved R18 235.0 mm to (61.2, 20.9)
- moved R19 224.0 mm to (68.1, 19.3)
- moved C36 216.8 mm to (47.6, 191.9)
- moved S0 216.8 mm to (87.8, 191.7)
- moved C24 215.1 mm to (42.4, 189.8)
- moved C23 214.6 mm to (42.4, 185.3)
- moved R4 209.9 mm to (128.7, 196.8)
- moved SS0 208.4 mm to (87.8, 191.7)
- moved C11 206.6 mm to (134.3, 191.7)
- moved R2 203.7 mm to (134.6, 196.8)
- moved R53 202.0 mm to (24.3, 104.4)
- moved SS8 200.1 mm to (87.8, 191.7)
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- renumbered J4 to J10, J15 to J3, J17 to J4, J16 to J5, J8 to J7, J10 to J8, J11 to J9
Connections:
- C1 pad 1: VCC -> +3V3
- C10 pad 2: VCC -> +3V3
- C17 pad 1: VCC -> +3V3
- C18 pad 2: VCC -> +3V3
- C19 pad 1: VCC -> +3V3
- C2 pad 1: VCC -> +3V3
- C3 pad 1: VCC -> +3V3
- C4 pad 1: VCC -> +3V3
- C6 pad 2: VCC -> +3V3
- C7 pad 2: VCC -> +3V3
- C8 pad 2: VCC -> +3V3
- C9 pad 2: VCC -> +3V3
- J10 pad 2: Net-(J4-Pad2) -> Net-(J10-Pad2)
- J10 pad 3: Net-(J4-Pad2) -> Net-(J10-Pad2)
- J3 pad 2: Net-(J15-Pad2) -> Net-(J3-Pad2)
- J3 pad 3: Net-(J15-Pad2) -> Net-(J3-Pad2)
- J4 pad 2: Net-(J17-Pad2) -> Net-(J4-Pad2)
- J4 pad 3: Net-(J17-Pad2) -> Net-(J4-Pad2)
- J5 pad 2: Net-(J16-Pad2) -> Net-(J5-Pad2)
- J5 pad 3: Net-(J16-Pad2) -> Net-(J5-Pad2)
- J7 pad 2: Net-(J8-Pad2) -> Net-(J7-Pad2)
- J7 pad 3: Net-(J8-Pad2) -> Net-(J7-Pad2)
- J8 pad 2: Net-(J10-Pad2) -> Net-(J8-Pad2)
- J8 pad 3: Net-(J10-Pad2) -> Net-(J8-Pad2)
- J9 pad 2: Net-(J11-Pad2) -> Net-(J9-Pad2)
- J9 pad 3: Net-(J11-Pad2) -> Net-(J9-Pad2)
- L1 pad 1: VCC -> +3V3
- L1 pad 2: VCC -> +3V3
- LED1 pad 2: VCC -> +3V3
- LED10 pad 2: VCC -> +3V3
- LED11 pad 2: VCC -> +3V3
- LED12 pad 2: VCC -> +3V3
- LED13 pad 2: VCC -> +3V3
- LED14 pad 2: VCC -> +3V3
- LED15 pad 2: VCC -> +3V3
- LED16 pad 2: VCC -> +3V3
- LED2 pad 2: VCC -> +3V3
- LED3 pad 2: VCC -> +3V3
- LED4 pad 2: VCC -> +3V3
- LED5 pad 2: VCC -> +3V3
- LED6 pad 2: VCC -> +3V3
- LED7 pad 2: VCC -> +3V3
- LED8 pad 2: VCC -> +3V3
- LED9 pad 2: VCC -> +3V3
- MCP2 pad 1: (no net) -> GATE_OUT1
- MCP2 pad 2: (no net) -> GATE_OUT2
- MCP2 pad 3: (no net) -> GATE_OUT3
- MCP2 pad 4: (no net) -> GATE_OUT4
- R2 pad 2: MIDI_OUT_INTERNAL -> (no net)
- U2 pad 1: MIDI_OUT_INTERNAL -> (no net)
- U3 pad 11: VCC -> +3V3
- U3 pad 12: VCC -> +3V3
- U3 pad 20: VCC -> +3V3
- U3 pad 31: VCC -> +3V3
- U3 pad 35: VCC -> +3V3
- U3 pad 41: VCC -> +3V3
- U3 pad 46: VCC -> +3V3
- U3 pad 47: VCC -> +3V3
- U3 pad 6: VCC -> +3V3
- U3 pad 7: Net-(C20-Pad1) -> (no net)
- U3 pad 8: VCC -> +3V3
Routing:
- net DAC0: track 0.00 -> 23.6 mm
- net DAC3: track 0.00 -> 23.1 mm
- net DAC7: track 0.00 -> 21.4 mm
- net DAC4: track 0.00 -> 20.9 mm
- net DAC6: track 0.00 -> 17.4 mm
- net DAC1: track 0.00 -> 17.0 mm
- net DAC5: track 0.00 -> 14.4 mm
- net DAC2: track 0.00 -> 14.4 mm
- net Net-(C28-Pad2): track 0.00 -> 10.2 mm
- net Net-(C31-Pad2): track 0.00 -> 10.2 mm
- net Net-(C34-Pad2): track 0.00 -> 10.1 mm
- net Net-(C30-Pad2): track 0.00 -> 9.83 mm
- net Net-(C27-Pad2): track 0.00 -> 8.98 mm
- net Net-(C32-Pad2): track 0.00 -> 8.90 mm
- net Net-(C29-Pad2): track 0.00 -> 8.90 mm
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- removed copper zone on F.Cu, net GND
Other:
- board size 116.2 x 110.5 mm -> 259.7 x 133.3 mm
- board text added: "PROTOTYPE #6 OCTOBER 2015"
- board text added: "ZETAOHM AFX-01 TENKAI KARIYA"
- board text removed: "ZETAOHM AFX-01 PROTOTYPE #5 TENKAI KARIYA JUNE 2015"
