File: afx-01_proto5.kicad_pcb (KiCad board)
At the start: 2 copper layers, 114.3 x 110.5 mm, 113 parts, among them J1 HeadphoneOut, J2 MicIn, P1 CONN_02X05, P2 CONN_02X05, U1 ADA_SSD1306_I2C, U2 Teensy_3.1, U3 SAM2695, U4 MicroSD_Adapter, X1 12MHz

Commit message: Moving on to proto6!
Parts:
- added U5: SSD1306, afx-01:SSD1306_XL, F.Cu at (137.2, 48.3)
- moved MCP2 224.7 mm to (102.6, 93.5)
- moved REF** 224.7 mm to (102.6, 93.5)
- moved SS5 222.7 mm to (106.7, 106.7)
- moved SS7 222.7 mm to (106.7, 116.8)
- moved SS4 222.7 mm to (98.4, 106.7)
- moved SS6 222.7 mm to (98.4, 116.8)
- moved R17 192.6 mm to (114.2, 83.2)
- moved R16 192.6 mm to (114.3, 79.4)
- moved MCP1 150.5 mm to (173.0, 132.9)
- moved REF** 150.5 mm to (173.0, 132.9)
- moved SS8 150.5 mm to (174.0, 123.2)
- moved SS9 150.5 mm to (174.0, 116.8)
- moved REF** 150.5 mm to (179.7, 138.4)
- moved LED12 120.2 mm to (159.5, 116.8)
- moved LED16 120.2 mm to (159.5, 131.1)
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Routing:
- net GND: track 658.2 -> 941.3 mm, vias 8 -> 14
- net (no net): track 262.9 -> 3.19 mm, vias 4 -> 0
- net VCC: track 598.7 -> 748.1 mm, vias 16 -> 18
- net /SwitchMatrix/SCL: track 3.25 -> 149.8 mm, vias 0 -> 2
- net /SwitchMatrix/SDA: track 14.7 -> 151.7 mm, vias 3 -> 4
- net Net-(MCP2-Pad23): track 6.60 -> 133.0 mm, vias 0 -> 1
- net Net-(MCP2-Pad27): track 6.60 -> 126.5 mm, vias 0 -> 1
- net AGND: track 93.3 -> 196.6 mm
- net Net-(ENC1-Pad4): track 0.00 -> 93.8 mm, vias 0 -> 1
- net /SoundBoard/MIDIIN: track 3.30 -> 93.2 mm
- net /SwitchMatrix/ENCB: track 2.71 -> 88.0 mm
- net /SwitchMatrix/ENCA: track 2.71 -> 84.7 mm
- net Net-(C20-Pad1): track 0.00 -> 82.0 mm, vias 0 -> 2
- net Net-(C11-Pad1): track 0.00 -> 77.7 mm, vias 0 -> 2
- net Net-(MCP1-Pad21): track 6.70 -> 80.2 mm, vias 0 -> 2
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Other:
- board size 114.3 x 110.5 mm -> 91.4 x 116.8 mm
