File: afx-01.kicad_pcb (KiCad board)
At the start: 2 copper layers, 114.3 x 110.5 mm, 113 parts, among them J1 HeadphoneOut, J2 MicIn, P1 CONN_02X05, P2 CONN_02X05, U1 ADA_SSD1306_I2C, U2 Teensy_3.1, U3 SAM2695, U4 MicroSD_Adapter, X1 12MHz

Commit message: BIG UPDATE! omg so big
New boards and other things.. jeesh it sbeen too long since the last update
Parts:
- removed the ENC1 at (262.9, 37.5)
- removed G***: LOGO, Logo:zetaOhmLogo
- removed G***: LOGO, Logo:small Logo Zetaohm
- removed REF** (x4): MountingHole_4mm, Mounting_Holes:MountingHole_4mm
- removed REF** (x3): Via, afx-01:Via
- removed SS4, SS8: DPST_Switch, afx-01:B3F-1050_6mm_Switch
- added ENC1: Encoder_switch, Zetaohm:AB2_ROTARY_ENCODER_W_SWITCH, F.Cu at (115.6, 35.8)
- added ENC1: Encoder_switch, Zetaohm:AB2_ROTARY_ENCODER_W_SWITCH, F.Cu at (135.3, 54.6)
- added J11: Mono_AudioConnector, Zetaohm:THONKICONN, F.Cu at (35.5, 127.2)
- added J11: Mono_AudioConnector, Zetaohm:THONKICONN, F.Cu at (36.2, 101.4)
- added J11: Mono_AudioConnector, Zetaohm:THONKICONN, F.Cu at (82.0, 115.0)
- added J12: Mono_AudioConnector, Zetaohm:THONKICONN, F.Cu at (38.4, 115.0)
- added J12: Mono_AudioConnector, Zetaohm:THONKICONN, F.Cu at (39.0, 89.2)
- added J12: Mono_AudioConnector, Zetaohm:THONKICONN, F.Cu at (77.8, 127.2)
- added J13: Mono_AudioConnector, Zetaohm:THONKICONN, F.Cu at (107.7, 127.2)
- added J14: Mono_AudioConnector, Zetaohm:THONKICONN, F.Cu at (54.6, 127.2)
- added J14: Mono_AudioConnector, Zetaohm:THONKICONN, F.Cu at (111.9, 115.0)
- added J18: Mono_AudioConnector, Zetaohm:THONKICONN, F.Cu at (44.8, 127.2)
- added J18: Mono_AudioConnector, Zetaohm:THONKICONN, F.Cu at (45.4, 101.4)
- added J18: Mono_AudioConnector, Zetaohm:THONKICONN, F.Cu at (72.7, 115.0)
- added J19: Mono_AudioConnector, Zetaohm:THONKICONN, F.Cu at (87.1, 127.2)
- added J20: Mono_AudioConnector, Zetaohm:THONKICONN, F.Cu at (117.0, 127.2)
- added J21: Mono_AudioConnector, Zetaohm:THONKICONN, F.Cu at (102.6, 115.0)
- added J4: Mono_AudioConnector, Zetaohm:THONKICONN, F.Cu at (91.2, 115.0)
- added J5: Mono_AudioConnector, Zetaohm:THONKICONN, F.Cu at (47.6, 115.0)
- added J5: Mono_AudioConnector, Zetaohm:THONKICONN, F.Cu at (48.3, 89.2)
- added J5: Mono_AudioConnector, Zetaohm:THONKICONN, F.Cu at (68.6, 127.2)
- added J6: Mono_AudioConnector, Zetaohm:THONKICONN, F.Cu at (98.5, 127.2)
- added J7: Mono_AudioConnector, Zetaohm:THONKICONN, F.Cu at (62.9, 115.0)
- added J7: Mono_AudioConnector, Zetaohm:THONKICONN, F.Cu at (121.1, 115.0)
- added J7: Mono_AudioConnector, Zetaohm:THONKICONN, F.Cu at (134.0, 34.9)
- added SS10: DPST_Switch, Zetaohm:B3F-1050_6mm_Switch, F.Cu at (119.8, 82.6)
- added SS11: DPST_Switch, Zetaohm:B3F-1050_6mm_Switch, F.Cu at (119.8, 96.6)
- added U6: DAC8718, Zetaohm:QFN-48-1EP_7x7mm_Pitch0.5mm, F.Cu at (41.3, 69.2)
- J1, J2: footprint afx-01:Switchcraft_3.5mm_SMD_Stereo -> Zetaohm:Switchcraft_3.5mm_SMD_Stereo
- LED1, LED10, LED11, LED12, LED13, LED14, LED15, LED16, LED2, LED3, LED4, LED5, LED6, LED7, LED8, LED9: footprint afx-01:WS2811_5mm_ThroughHole -> Zetaohm:WS2812b_SMD
- S1, S10, S11, S12, S13, S14, S15, S16, S2, S3, S4, S5, S6, S7, S8, S9, SS1, SS2, SS3, SS5, SS6, SS7, SS9: footprint afx-01:B3F-1050_6mm_Switch -> Zetaohm:B3F-1050_6mm_Switch
- U1: footprint ab2_header:AB2_HDR_M08-1V -> Zetaohm:SSD1306
- U2: footprint afx-01:Teensy3.1 -> Zetaohm:Teensy3.1; moved to F.Cu
- U4: footprint afx-01:MicroSD -> Zetaohm:MicroSD
- X1: footprint afx-01:Xtal_3.2mm -> Zetaohm:Xtal_3.2mm
- moved SS5 270.2 mm to (57.7, 68.6), turned to 0 degrees
- moved SS7 270.1 mm to (57.7, 96.6), turned to 0 degrees
- moved SS6 261.8 mm to (57.7, 82.6), turned to 0 degrees
- moved MCP1 235.8 mm to (88.9, 89.4)
- moved MCP2 235.6 mm to (89.2, 61.2)
- moved SS9 206.9 mm to (119.8, 68.6)
- moved C26 182.0 mm to (59.5, 26.2), turned to 180 degrees
- moved C25 181.2 mm to (59.5, 28.7), turned to 0 degrees
- moved R3 181.2 mm to (59.0, 33.3), turned to 180 degrees
- moved D1 180.8 mm to (59.0, 35.8), turned to 0 degrees
- moved C5 180.1 mm to (59.2, 38.4), turned to 180 degrees
- moved LED14 175.6 mm to (75.8, 103.6), turned to 90 degrees
- moved LED13 175.6 mm to (61.8, 103.6), turned to 90 degrees
- moved LED10 175.6 mm to (75.8, 89.6), turned to 90 degrees
- moved LED9 175.6 mm to (61.8, 89.6), turned to 90 degrees
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Connections:
- LED10 pad 1: Net-(LED10-Pad1) -> Net-(LED1-Pad1)
- LED10 pad 4: Net-(LED10-Pad4) -> Net-(LED1-Pad4)
- LED11 pad 1: Net-(LED10-Pad4) -> Net-(LED1-Pad1)
- LED11 pad 4: Net-(LED11-Pad4) -> Net-(LED1-Pad4)
- LED12 pad 1: Net-(LED11-Pad4) -> Net-(LED1-Pad1)
- LED12 pad 4: Net-(LED12-Pad4) -> Net-(LED1-Pad4)
- LED13 pad 1: Net-(LED12-Pad4) -> Net-(LED1-Pad1)
- LED13 pad 4: Net-(LED13-Pad4) -> Net-(LED1-Pad4)
- LED14 pad 1: Net-(LED13-Pad4) -> Net-(LED1-Pad1)
- LED14 pad 4: Net-(LED14-Pad4) -> Net-(LED1-Pad4)
- LED15 pad 1: Net-(LED14-Pad4) -> Net-(LED1-Pad1)
- LED15 pad 4: Net-(LED15-Pad4) -> Net-(LED1-Pad4)
- LED16 pad 1: Net-(LED15-Pad4) -> Net-(LED1-Pad1)
- LED16 pad 4: (no net) -> Net-(LED1-Pad4)
- LED2 pad 1: Net-(LED1-Pad4) -> Net-(LED1-Pad1)
- LED2 pad 4: Net-(LED2-Pad4) -> Net-(LED1-Pad4)
- LED3 pad 1: Net-(LED2-Pad4) -> Net-(LED1-Pad1)
- LED3 pad 4: Net-(LED3-Pad4) -> Net-(LED1-Pad4)
- LED4 pad 1: Net-(LED3-Pad4) -> Net-(LED1-Pad1)
- LED4 pad 4: Net-(LED4-Pad4) -> Net-(LED1-Pad4)
- LED5 pad 1: Net-(LED4-Pad4) -> Net-(LED1-Pad1)
- LED5 pad 4: Net-(LED5-Pad4) -> Net-(LED1-Pad4)
- LED6 pad 1: Net-(LED5-Pad4) -> Net-(LED1-Pad1)
- LED6 pad 4: Net-(LED6-Pad4) -> Net-(LED1-Pad4)
- LED7 pad 1: Net-(LED6-Pad4) -> Net-(LED1-Pad1)
- LED7 pad 4: Net-(LED7-Pad4) -> Net-(LED1-Pad4)
- LED8 pad 1: Net-(LED7-Pad4) -> Net-(LED1-Pad1)
- LED8 pad 4: Net-(LED8-Pad4) -> Net-(LED1-Pad4)
- LED9 pad 1: Net-(LED8-Pad4) -> Net-(LED1-Pad1)
- LED9 pad 4: Net-(LED10-Pad1) -> Net-(LED1-Pad4)
- S10 pad 1: Net-(MCP1-Pad23) -> Net-(MCP1-Pad17)
- S10 pad 2: Net-(MCP1-Pad23) -> Net-(MCP1-Pad17)
- S11 pad 1: Net-(MCP1-Pad27) -> Net-(MCP1-Pad17)
- S11 pad 2: Net-(MCP1-Pad27) -> Net-(MCP1-Pad17)
- S12 pad 1: Net-(MCP1-Pad3) -> Net-(MCP1-Pad17)
- S12 pad 2: Net-(MCP1-Pad3) -> Net-(MCP1-Pad17)
- S13 pad 1: Net-(MCP1-Pad20) -> Net-(MCP1-Pad17)
- S13 pad 2: Net-(MCP1-Pad20) -> Net-(MCP1-Pad17)
- S14 pad 1: Net-(MCP1-Pad24) -> Net-(MCP1-Pad17)
- S14 pad 2: Net-(MCP1-Pad24) -> Net-(MCP1-Pad17)
- S15 pad 1: Net-(MCP1-Pad28) -> Net-(MCP1-Pad17)
- S15 pad 2: Net-(MCP1-Pad28) -> Net-(MCP1-Pad17)
- S16 pad 1: Net-(MCP1-Pad4) -> Net-(MCP1-Pad17)
- S16 pad 2: Net-(MCP1-Pad4) -> Net-(MCP1-Pad17)
- S2 pad 1: Net-(MCP1-Pad21) -> Net-(MCP1-Pad17)
- S2 pad 2: Net-(MCP1-Pad21) -> Net-(MCP1-Pad17)
- S3 pad 1: Net-(MCP1-Pad25) -> Net-(MCP1-Pad17)
- S3 pad 2: Net-(MCP1-Pad25) -> Net-(MCP1-Pad17)
- S4 pad 1: Net-(MCP1-Pad1) -> Net-(MCP1-Pad17)
- S4 pad 2: Net-(MCP1-Pad1) -> Net-(MCP1-Pad17)
- S5 pad 1: Net-(MCP1-Pad18) -> Net-(MCP1-Pad17)
- S5 pad 2: Net-(MCP1-Pad18) -> Net-(MCP1-Pad17)
- S6 pad 1: Net-(MCP1-Pad22) -> Net-(MCP1-Pad17)
- S6 pad 2: Net-(MCP1-Pad22) -> Net-(MCP1-Pad17)
- S7 pad 1: Net-(MCP1-Pad26) -> Net-(MCP1-Pad17)
- S7 pad 2: Net-(MCP1-Pad26) -> Net-(MCP1-Pad17)
- S8 pad 1: Net-(MCP1-Pad2) -> Net-(MCP1-Pad17)
- S8 pad 2: Net-(MCP1-Pad2) -> Net-(MCP1-Pad17)
- S9 pad 1: Net-(MCP1-Pad19) -> Net-(MCP1-Pad17)
- S9 pad 2: Net-(MCP1-Pad19) -> Net-(MCP1-Pad17)
- SS2 pad 1: Net-(MCP2-Pad21) -> Net-(MCP2-Pad17)
- SS2 pad 2: Net-(MCP2-Pad21) -> Net-(MCP2-Pad17)
- SS3 pad 1: Net-(MCP2-Pad25) -> Net-(MCP2-Pad17)
- SS3 pad 2: Net-(MCP2-Pad25) -> Net-(MCP2-Pad17)
- SS5 pad 1: Net-(MCP2-Pad22) -> Net-(MCP2-Pad17)
- SS5 pad 2: Net-(MCP2-Pad22) -> Net-(MCP2-Pad17)
- SS6 pad 1: Net-(MCP2-Pad26) -> Net-(MCP2-Pad17)
- SS6 pad 2: Net-(MCP2-Pad26) -> Net-(MCP2-Pad17)
- SS7 pad 1: Net-(MCP2-Pad19) -> Net-(MCP2-Pad17)
- SS7 pad 2: Net-(MCP2-Pad19) -> Net-(MCP2-Pad17)
- SS9 pad 1: Net-(MCP2-Pad27) -> Net-(MCP2-Pad17)
- SS9 pad 2: Net-(MCP2-Pad27) -> Net-(MCP2-Pad17)
- U1 pad 6: (no net) -> Net-(U1-Pad6)
- X1 pad 2: GND -> (no net)
Routing:
- net GND: track 658.2 -> 0.00 mm, vias 8 -> 0
- net VCC: track 598.7 -> 0.00 mm, vias 16 -> 0
- net (no net): track 262.9 -> 0.00 mm, vias 4 -> 0
- net Net-(MCP1-Pad19): track 94.5 -> 0.00 mm, vias 2 -> 0
- net AGND: track 93.3 -> 0.00 mm, vias 4 -> 0
- net Net-(MCP1-Pad17): track 91.3 -> 0.00 mm, vias 2 -> 0
- net /29: track 85.6 -> 0.00 mm, vias 2 -> 0
- net Net-(MCP1-Pad18): track 79.6 -> 0.00 mm, vias 1 -> 0
- net /30: track 79.4 -> 0.00 mm
- net Net-(MCP1-Pad20): track 76.3 -> 0.00 mm
- net Net-(MCP1-Pad22): track 65.8 -> 0.00 mm, vias 1 -> 0
- net Net-(LED4-Pad4): track 62.7 -> 0.00 mm
- net Net-(MCP1-Pad23): track 60.4 -> 0.00 mm, vias 1 -> 0
- net Net-(MCP1-Pad24): track 58.7 -> 0.00 mm
- net Net-(LED8-Pad4): track 55.5 -> 0.00 mm
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Other:
- board size 114.3 x 110.5 mm -> 116.2 x 110.5 mm
