File: afx-01.kicad_pcb (KiCad board)
At the start: 2 copper layers, 116.2 x 110.5 mm, 198 parts, among them J1 HeadphoneOut, J10 Mono_AudioConnector, J11 Mono_AudioConnector, J12 Mono_AudioConnector, J13 Mono_AudioConnector, J14 Mono_AudioConnector, J15 Mono_AudioConnector, J16 Mono_AudioConnector, J17 Mono_AudioConnector, J18 Mono_AudioConnector, J2 MicIn, J3 Mono_AudioConnector, J4 Mono_AudioConnector, J5 Mono_AudioConnector, J6 Mono_AudioConnector, J7 Mono_AudioConnector, J8 Mono_AudioConnector, J9 Mono_AudioConnector, P1 CONN_02X05, P2 CONN_02X05, Q1 Q_NPN_BCE, Q2 Q_NPN_BCE, Q3 Q_NPN_BCE, Q4 Q_NPN_BCE, U1 ADA_SSD1306_I2C, U13 MCP6004, U2 Teensy_3.1, U3 SAM2695, U4 MicroSD_Adapter, U5 MCP1703, U6 OPA4171, U7 OPA4171, U8 AD5676, X1 12MHz

Commit message: Added Touch Capacitive Panel
Parts:
- removed C20: 1µfT, Capacitors_SMD:C_0805_HandSoldering
- removed C21: 220pF, Capacitors_SMD:C_0805_HandSoldering
- removed J1: HeadphoneOut, Zetaohm:Switchcraft_3.5mm_SMD_Stereo
- removed J2: MicIn, Zetaohm:Switchcraft_3.5mm_SMD_Stereo
- removed the J3 at (88.6, 143.4)
- removed the J5 at (88.6, 143.4)
- removed the J7 at (88.6, 143.4)
- removed the J9 at (88.6, 143.4)
- removed R7: 4.7k, Resistors_SMD:R_0805_HandSoldering
- added G***: CAPACITIVE_FACEPLATE, Zetaohm:FACEPLATEV1, F.Cu at (213.3, 91.2)
- added J11: Mono_AudioConnector, Zetaohm:THONKICONN, F.Cu at (24.8, 139.3)
- added J15: Mono_AudioConnector, Zetaohm:THONKICONN, F.Cu at (44.9, 127.6)
- added J16: Mono_AudioConnector, Zetaohm:THONKICONN, F.Cu at (54.4, 127.6)
- added J17: Mono_AudioConnector, Zetaohm:THONKICONN, F.Cu at (43.6, 139.3)
- added J19: Mono_AudioConnector, Zetaohm:THONKICONN, F.Cu at (82.7, 127.6)
- added J20: Mono_AudioConnector, Zetaohm:THONKICONN, F.Cu at (81.2, 139.3)
- added J21: Mono_AudioConnector, Zetaohm:THONKICONN, F.Cu at (120.4, 127.6)
- added J21: Mono_AudioConnector, Zetaohm:THONKICONN, F.Cu at (111.0, 127.6)
- added J22: Mono_AudioConnector, Zetaohm:THONKICONN, F.Cu at (109.5, 139.3)
- added JP3: JUMPER3, Zetaohm:Jumper_3way, F.Cu at (121.7, 67.8)
- added LED17: WS2812b, Zetaohm:WS2812b_SMD, F.Cu at (54.8, 114.5)
- added LED18: WS2812b, Zetaohm:WS2812b_SMD, F.Cu at (72.2, 114.5)
- added LED19: WS2812b, Zetaohm:WS2812b_SMD, F.Cu at (89.6, 114.5)
- added LED20: WS2812b, Zetaohm:WS2812b_SMD, F.Cu at (107.0, 114.5)
- added Q5: BSS138, Housings_SOT-23_SOT-143_TSOT-6:SOT-23, F.Cu at (125.2, 78.0)
- added Q6: BSS138, Housings_SOT-23_SOT-143_TSOT-6:SOT-23, F.Cu at (126.2, 86.2)
- added R72: 4.7k, Resistors_SMD:R_0603_HandSoldering, F.Cu at (118.6, 85.7)
- added R73: 4.7k, Resistors_SMD:R_0603_HandSoldering, F.Cu at (118.6, 92.6)
- added R74: 1k, Resistors_SMD:R_0603_HandSoldering, F.Cu at (56.5, 191.9)
- added R75: 1k, Resistors_SMD:R_0603_HandSoldering, F.Cu at (52.1, 191.9)
- added R76: 1k, Resistors_SMD:R_0603_HandSoldering, F.Cu at (56.5, 186.0)
- added R77: 1k, Resistors_SMD:R_0603_HandSoldering, F.Cu at (52.1, 186.0)
- added U10: MicroSD_Connector, Zetaohm:AMPHENOL_MICROSD, F.Cu at (104.2, 11.4)
- added U9: 3_pin_stereo, Zetaohm:KOBICONN_ST, F.Cu at (118.6, 139.3)
- C1, C2, C3, C4: value 100µf -> 100uf; footprint Capacitors_SMD:C_0805_HandSoldering -> Capacitors_SMD:C_0603_HandSoldering
- C10, C11, C12, C13, C14, C15, C16, C17, C18, C19, C22, C23, C24, C25, C26, C27, C28, C29, C30, C31, C32, C33, C34, C35, C36, C37, C38, C39, C40, C5, C6, C7, C8, C9, L1: footprint Capacitors_SMD:C_0805_HandSoldering -> Capacitors_SMD:C_0603_HandSoldering
- MIDI_IN1, MIDI_OUT1: moved to F.Cu
- P2: value CONN_02X05 -> CONN_02X08; footprint ab2_header:AB2_HDR_M05-2V -> Pin_Headers:Pin_Header_Straight_2x08; moved to F.Cu
- Q1, Q2, Q3, Q4: value Q_NPN_BCE -> BSS138
- R1, R10, R11, R12, R13, R14, R15, R16, R17, R18, R19, R2, R20, R21, R22, R23, R24, R25, R26, R27, R28, R29, R3, R30, R31, R32, R33, R34, R35, R36, R37, R38, R39, R4, R40, R41, R42, R43, R44, R45, R46, R47, R48, R49, R5, R50, R51, R52, R53, R54, R55, R56, R57, R58, R59, R6, R60, R61, R62, R63, R64, R65, R66, R67, R68, R69, R70, R71, R8, R9: footprint Resistors_SMD:R_0805_HandSoldering -> Resistors_SMD:R_0603_HandSoldering
- U2: footprint Zetaohm:Teensy3.1 -> Zetaohm:Teensy3.1_Min_I2C2
- moved R56 264.5 mm to (24.3, 106.3), turned to 180 degrees
- moved R57 258.5 mm to (35.8, 106.2), turned to 180 degrees
- moved Q1 249.8 mm to (23.8, 109.1), turned to 90 degrees
- moved R66 247.7 mm to (37.0, 87.8), turned to 180 degrees
- moved R65 241.8 mm to (37.0, 89.5)
- moved C37 240.9 mm to (42.1, 74.9)
- moved R61 240.0 mm to (47.4, 104.4)
- moved C36 238.4 mm to (47.6, 191.9)
- moved C40 238.1 mm to (41.9, 86.0)
- moved R68 238.0 mm to (41.9, 89.5), turned to 180 degrees
- moved R54 237.6 mm to (35.8, 104.4)
- moved Q3 236.7 mm to (46.8, 109.1), turned to 90 degrees
- moved R67 236.4 mm to (37.0, 91.3)
- moved R59 234.5 mm to (37.1, 73.2), turned to 180 degrees
- moved R62 233.6 mm to (59.3, 104.4)
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- renumbered J4 to J10, J15 to J3, J17 to J4, J16 to J5, J8 to J7, J10 to J8, J11 to J9
Connections:
- C1 pad 1: VCC -> +3V3
- C10 pad 2: VCC -> +3V3
- C17 pad 1: VCC -> +3V3
- C18 pad 2: VCC -> +3V3
- C19 pad 1: VCC -> +3V3
- C2 pad 1: VCC -> +3V3
- C3 pad 1: VCC -> +3V3
- C4 pad 1: VCC -> +3V3
- C6 pad 2: VCC -> +3V3
- C7 pad 2: VCC -> +3V3
- C8 pad 2: VCC -> +3V3
- C9 pad 2: VCC -> +3V3
- J10 pad 2: Net-(J4-Pad2) -> Net-(J10-Pad2)
- J10 pad 3: Net-(J4-Pad2) -> Net-(J10-Pad2)
- J3 pad 2: Net-(J15-Pad2) -> Net-(J3-Pad2)
- J3 pad 3: Net-(J15-Pad2) -> Net-(J3-Pad2)
- J4 pad 2: Net-(J17-Pad2) -> Net-(J4-Pad2)
- J4 pad 3: Net-(J17-Pad2) -> Net-(J4-Pad2)
- J5 pad 2: Net-(J16-Pad2) -> Net-(J5-Pad2)
- J5 pad 3: Net-(J16-Pad2) -> Net-(J5-Pad2)
- J7 pad 2: Net-(J8-Pad2) -> Net-(J7-Pad2)
- J7 pad 3: Net-(J8-Pad2) -> Net-(J7-Pad2)
- J8 pad 2: Net-(J10-Pad2) -> Net-(J8-Pad2)
- J8 pad 3: Net-(J10-Pad2) -> Net-(J8-Pad2)
- J9 pad 2: Net-(J11-Pad2) -> Net-(J9-Pad2)
- J9 pad 3: Net-(J11-Pad2) -> Net-(J9-Pad2)
- L1 pad 1: VCC -> +3V3
- L1 pad 2: VCC -> +3V3
- LED1 pad 2: VCC -> +3V3
- LED10 pad 2: VCC -> +3V3
- LED11 pad 2: VCC -> +3V3
- LED12 pad 2: VCC -> +3V3
- LED13 pad 2: VCC -> +3V3
- LED14 pad 2: VCC -> +3V3
- LED15 pad 2: VCC -> +3V3
- LED16 pad 2: VCC -> +3V3
- LED2 pad 2: VCC -> +3V3
- LED3 pad 2: VCC -> +3V3
- LED4 pad 2: VCC -> +3V3
- LED5 pad 2: VCC -> +3V3
- LED6 pad 2: VCC -> +3V3
- LED7 pad 2: VCC -> +3V3
- LED8 pad 2: VCC -> +3V3
- LED9 pad 2: VCC -> +3V3
- MCP1 pad 8: SCL0 -> SCL0_5v
- MCP1 pad 9: SDA0 -> SDA0_5v
- MCP2 pad 1: (no net) -> GATE_OUT1
- MCP2 pad 2: (no net) -> GATE_OUT2
- MCP2 pad 3: (no net) -> GATE_OUT3
- MCP2 pad 4: (no net) -> GATE_OUT4
- MCP2 pad 8: SCL0 -> SCL0_5v
- MCP2 pad 9: SDA0 -> SDA0_5v
- R2 pad 2: MIDI_OUT_INTERNAL -> (no net)
- U2 pad 1: MIDI_OUT_INTERNAL -> (no net)
- U3 pad 11: VCC -> +3V3
- U3 pad 12: VCC -> +3V3
- U3 pad 20: VCC -> +3V3
- U3 pad 31: VCC -> +3V3
- U3 pad 35: VCC -> +3V3
- U3 pad 41: VCC -> +3V3
- U3 pad 46: VCC -> +3V3
- U3 pad 47: VCC -> +3V3
- U3 pad 6: VCC -> +3V3
- U3 pad 7: Net-(C20-Pad1) -> (no net)
- U3 pad 8: VCC -> +3V3
- U5 pad 2: +5V -> Net-(JP3-Pad1)
Routing:
- net DAC0: track 0.00 -> 23.6 mm
- net DAC3: track 0.00 -> 23.1 mm
- net DAC7: track 0.00 -> 21.4 mm
- net DAC4: track 0.00 -> 20.9 mm
- net DAC6: track 0.00 -> 17.4 mm
- net DAC1: track 0.00 -> 17.0 mm
- net DAC5: track 0.00 -> 14.4 mm
- net DAC2: track 0.00 -> 14.4 mm
- net Net-(C28-Pad2): track 0.00 -> 10.2 mm
- net Net-(C31-Pad2): track 0.00 -> 10.2 mm
- net Net-(C34-Pad2): track 0.00 -> 10.1 mm
- net Net-(C30-Pad2): track 0.00 -> 9.83 mm
- net Net-(C27-Pad2): track 0.00 -> 8.98 mm
- net Net-(C32-Pad2): track 0.00 -> 8.90 mm
- net Net-(C29-Pad2): track 0.00 -> 8.90 mm
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- removed copper zone on F.Cu, net GND
Other:
- board size 116.2 x 110.5 mm -> 259.7 x 133.3 mm
- board text added: "PROTOTYPE #6 OCTOBER 2015"
- board text added: "ZETAOHM AFX-01 TENKAI KARIYA"
- board text removed: "ZETAOHM AFX-01 PROTOTYPE #5 TENKAI KARIYA JUNE 2015"
