File: afx-01.kicad_pcb (KiCad board)
At the start: 2 copper layers, 259.7 x 133.3 mm, 214 parts, among them J10 Mono_AudioConnector, J11 Mono_AudioConnector, J12 Mono_AudioConnector, J13 Mono_AudioConnector, J14 Mono_AudioConnector, J15 Mono_AudioConnector, J16 Mono_AudioConnector, J17 Mono_AudioConnector, J18 Mono_AudioConnector, J19 Mono_AudioConnector, J20 Mono_AudioConnector, J21 Mono_AudioConnector, J22 Mono_AudioConnector, J3 Mono_AudioConnector, J4 Mono_AudioConnector, J5 Mono_AudioConnector, J6 Mono_AudioConnector, J7 Mono_AudioConnector, J8 Mono_AudioConnector, J9 Mono_AudioConnector, P1 CONN_02X05, P2 CONN_02X08, Q1 BSS138, Q2 BSS138, Q3 BSS138, Q4 BSS138, Q5 BSS138, Q6 BSS138, U1 ADA_SSD1306_I2C, U10 MicroSD_Connector, U13 MCP6004, U2 Teensy_3.1, U3 SAM2695, U4 MicroSD_Adapter, U5 MCP1703, U6 OPA4171, U7 OPA4171, U8 AD5676, U9 3_pin_stereo, X1 12MHz

Commit message: Updating footprints
Parts:
- removed ENC2: Encoder_switch, Zetaohm:AB2_ROTARY_ENCODER_W_SWITCH
- removed G***: CAPACITIVE_FACEPLATE, Zetaohm:FACEPLATEV1
- removed J21 (x2), J22: Mono_AudioConnector, Zetaohm:THONKICONN
- removed MCP2: MCP23017-QFN, Housings_DFN_QFN:QFN-28-1EP_6x6mm_Pitch0.65mm
- removed S0, S1, S10, S11, S12, S13, S14, S15, S2, S3, S4, S5, S6, S7, S8, S9, SS0, SS1, SS2, SS3, SS4, SS5, SS6, SS7, SS8: DPST_Switch, Zetaohm:B3F-1050_6mm_Switch
- added C20: .01µf, Capacitors_SMD:C_0603_HandSoldering, F.Cu at (185.6, 73.0)
- added C21: .01µf, Capacitors_SMD:C_0603_HandSoldering, F.Cu at (180.4, 78.9)
- added C41: 0.1uf, Capacitors_SMD:C_0603_HandSoldering, F.Cu at (184.9, 78.9)
- added C42: 0.1uf, Capacitors_SMD:C_0603_HandSoldering, F.Cu at (180.3, 84.8)
- added C43: 0.1uf, Capacitors_SMD:C_0603_HandSoldering, F.Cu at (190.1, 73.0)
- added C44: 0.1uf, Capacitors_SMD:C_0603_HandSoldering, F.Cu at (204.3, 60.8)
- added C45: 4.7nf, Capacitors_SMD:C_0603_HandSoldering, F.Cu at (194.5, 76.4)
- added C46: 18pf, Capacitors_SMD:C_0603_HandSoldering, F.Cu at (208.5, 60.8)
- added C47: 4.7nf, Capacitors_SMD:C_0603_HandSoldering, F.Cu at (204.3, 66.7)
- added C48: 18pf, Capacitors_SMD:C_0603_HandSoldering, F.Cu at (189.2, 78.9)
- added C49: 4.7nf, Capacitors_SMD:C_0603_HandSoldering, F.Cu at (184.7, 84.8)
- added C50: 4.7nf, Capacitors_SMD:C_0603_HandSoldering, F.Cu at (180.3, 90.7)
- added C51: 4.7nf, Capacitors_SMD:C_0603_HandSoldering, F.Cu at (193.4, 82.3)
- added C52: 4.7nf, Capacitors_SMD:C_0603_HandSoldering, F.Cu at (184.7, 90.7)
- added J1: Mono_AudioConnector, Zetaohm:THONKICONN, F.Cu at (220.8, 94.0)
- added J2: Mono_AudioConnector, Zetaohm:THONKICONN, F.Cu at (220.8, 111.8)
- added JP4: JUMPER3, Zetaohm:Jumper_3way, F.Cu at (182.7, 121.1)
- added JP5: JUMPER3, Zetaohm:Jumper_3way, F.Cu at (200.5, 100.2)
- added JP6: JUMPER3, Zetaohm:Jumper_3way, F.Cu at (262.1, 90.1)
- added JP7: JUMPER3, Zetaohm:Jumper_3way, F.Cu at (249.4, 100.9)
- added R7: 1k, Resistors_SMD:R_0603_HandSoldering, F.Cu at (260.8, 96.3)
- added R78: 1k, Resistors_SMD:R_0603_HandSoldering, F.Cu at (212.8, 60.8)
- added R79: 1k, Resistors_SMD:R_0603_HandSoldering, F.Cu at (208.7, 66.7)
- added R80: 1k, Resistors_SMD:R_0603_HandSoldering, F.Cu at (221.7, 60.8)
- added R81: 1k, Resistors_SMD:R_0603_HandSoldering, F.Cu at (207.8, 78.5)
- added R82: 1k, Resistors_SMD:R_0603_HandSoldering, F.Cu at (198.1, 88.2)
- added R83: 470k, Resistors_SMD:R_0603_HandSoldering, F.Cu at (217.6, 66.7)
- added R84: 470k, Resistors_SMD:R_0603_HandSoldering, F.Cu at (212.3, 72.6)
- added R85: 470k, Resistors_SMD:R_0603_HandSoldering, F.Cu at (202.5, 84.4)
- added R86: 470k, Resistors_SMD:R_0603_HandSoldering, F.Cu at (226.2, 60.8)
- added R87: 470k, Resistors_SMD:R_0603_HandSoldering, F.Cu at (207.0, 84.4)
- added R88: 470k, Resistors_SMD:R_0603_HandSoldering, F.Cu at (216.7, 72.6)
- added RP1: 10k, Resistors_SMD:R_0603_HandSoldering, F.Cu at (181.1, 73.0)
- added U11: MCP1703, Housings_SOT-23_SOT-143_TSOT-6:SOT-23_Handsoldering, F.Cu at (198.3, 62.7)
- added U12: QT1481, Housings_QFP:LQFP-44_10x10mm_Pitch0.8mm, F.Cu at (167.6, 47.0)
- added X2: 16Mhz, Crystals:Crystal_HC49-SD_SMD, F.Cu at (186.7, 63.9)
- C23, C24, C35, C36: value .01µf -> 0.1uf
- L1: footprint Capacitors_SMD:C_0603_HandSoldering -> Capacitors_SMD:C_0805_HandSoldering
- MIDI_OPTOISOLATOR1: footprint Housings_DIP:DIP-8__300_ELL -> SMD_Packages:DIP-8_SMD
- MIDI_OUT1: footprint Zetaohm:MIDI_Wire_Connector -> SMD_Packages:DIP-8_SMD
- P2: footprint Pin_Headers:Pin_Header_Straight_2x08 -> Pin_Headers:Pin_Header_Angled_2x08
- R12, R13, R14, R15, R47, R48, R49, R50: value 10k -> 1k
- U1: footprint Zetaohm:SSD1306 -> Pin_Headers:Pin_Header_Angled_1x06
- moved R74 192.7 mm to (207.8, 72.6)
- moved C36 192.4 mm to (196.8, 70.5)
- moved R76 185.6 mm to (203.4, 72.6)
- moved C24 184.1 mm to (206.6, 106.4), turned to 0 degrees
- moved R77 183.3 mm to (198.9, 76.4)
- moved JP2 176.8 mm to (200.5, 106.5)
- moved JP1 175.1 mm to (207.9, 100.2)
- moved C23 172.7 mm to (199.2, 112.8), turned to 0 degrees
- moved R75 171.9 mm to (189.2, 88.2)
- moved R13 163.2 mm to (268.1, 90.0), turned to 0 degrees
- moved J20 158.7 mm to (237.5, 111.8), turned to 0 degrees
- moved J19 158.1 mm to (237.5, 95.7)
- moved C35 155.4 mm to (188.7, 121.0)
- moved R12 154.3 mm to (255.5, 100.8), turned to 0 degrees
- moved R18 150.6 mm to (172.8, 122.0)
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- renumbered LED20 to LED1
Connections:
- C23 pad 1: ENC2A -> GND
- C23 pad 2: GND -> Net-(C23-Pad2)
- C24 pad 1: ENC2B -> Net-(C24-Pad1)
- C35 pad 1: ENC1A -> VDD
- C36 pad 1: ENC1B -> Net-(C36-Pad1)
- ENC1 pad 1: Net-(ENC1-Pad1) -> (no net)
- ENC1 pad 3: Net-(ENC1-Pad3) -> (no net)
- JP3 pad 1: Net-(JP3-Pad1) -> Net-(C24-Pad1)
- JP3 pad 3: Net-(JP3-Pad3) -> Net-(C23-Pad2)
- MCP1 pad 1: SC -> (no net)
- MCP1 pad 11: GND -> +5V
- MCP1 pad 14: VCC -> +5V
- MCP1 pad 17: S0 -> MCP_GATE_IN1
- MCP1 pad 18: S1 -> MCP_GATE_IN2
- MCP1 pad 19: S2 -> MCP_GATE_IN3
- MCP1 pad 2: SD -> (no net)
- MCP1 pad 20: S3 -> MCP_GATE_IN4
- MCP1 pad 21: S4 -> GATE_OUT1
- MCP1 pad 22: S5 -> GATE_OUT2
- MCP1 pad 23: S6 -> GATE_OUT3
- MCP1 pad 24: S7 -> GATE_OUT4
- MCP1 pad 25: S8 -> ENC1SW
- MCP1 pad 26: S9 -> (no net)
- MCP1 pad 27: SA -> (no net)
- MCP1 pad 28: SB -> (no net)
- MCP1 pad 3: SE -> (no net)
- MCP1 pad 4: SF -> (no net)
- MCP1 pad 5: VCC -> +5V
- P2 pad 11: Net-(JP3-Pad3) -> Net-(C23-Pad2)
- P2 pad 12: Net-(JP3-Pad3) -> Net-(C23-Pad2)
- Q1 pad 2: GATE_IN1 -> MCP_GATE_IN1
- Q2 pad 2: GATE_IN2 -> MCP_GATE_IN2
- R12 pad 1: Net-(ENC2-Pad1) -> Net-(J2-Pad2)
- R12 pad 2: ENC2A -> GATE_OUT2
- R13 pad 1: Net-(ENC2-Pad1) -> Net-(J19-Pad2)
- R13 pad 2: VCC -> GATE_OUT3
- R14 pad 1: Net-(ENC2-Pad3) -> Net-(J20-Pad2)
- R14 pad 2: VCC -> GATE_OUT4
- R15 pad 1: Net-(ENC2-Pad3) -> (no net)
- R15 pad 2: ENC2B -> Net-(R15-Pad2)
- R2 pad 2: (no net) -> MIDI_OUT_EXTERNAL
- R47 pad 1: Net-(ENC1-Pad1) -> (no net)
- R47 pad 2: ENC1A -> Net-(R47-Pad2)
- R48 pad 1: Net-(ENC1-Pad1) -> (no net)
- R48 pad 2: VCC -> Net-(R48-Pad2)
- R49 pad 1: Net-(ENC1-Pad3) -> (no net)
- R49 pad 2: VCC -> Net-(R49-Pad2)
- R50 pad 1: Net-(ENC1-Pad3) -> (no net)
- R50 pad 2: ENC1B -> Net-(R50-Pad2)
- R53 pad 2: GATE_IN1 -> MCP_GATE_IN1
- R54 pad 2: GATE_IN2 -> MCP_GATE_IN2
- R74 pad 1: Net-(J19-Pad2) -> (no net)
- R74 pad 2: GATE_OUT1 -> Net-(R74-Pad2)
- R75 pad 1: Net-(J20-Pad2) -> (no net)
- R75 pad 2: GATE_OUT2 -> Net-(R75-Pad2)
- R76 pad 1: Net-(J21-Pad2) -> (no net)
- R76 pad 2: GATE_OUT3 -> Net-(R76-Pad2)
- R77 pad 1: Net-(J22-Pad2) -> (no net)
- R77 pad 2: GATE_OUT4 -> Net-(C45-Pad1)
- U1 pad 6: Net-(U1-Pad6) -> (no net)
- U2 pad 0: GATE_IN1 -> (no net)
- U2 pad 10: SD_CS -> QT_RX
- U2 pad 14: ENC2B -> GATE_IN3
- U2 pad 15: ENC2A -> GATE_IN4
- U2 pad 2: GATE_IN2 -> SD_CS
- U2 pad 3: GATE_IN3 -> DAC_CS
- U2 pad 4: GATE_IN4 -> (no net)
- U2 pad 41: (no net) -> QT_CS
- U2 pad 9: DAC_CS -> QT_TX
- U5 pad 2: Net-(JP3-Pad1) -> Net-(C24-Pad1)
