File: afx-01_proto5 2.kicad_pcb (KiCad board)
At the start: 2 copper layers, 114.3 x 110.5 mm, 113 parts, among them J1 HeadphoneOut, J2 MicIn, P1 CONN_02X05, P2 CONN_02X05, U1 ADA_SSD1306_I2C, U2 Teensy_3.1, U3 SAM2695, U4 MicroSD_Adapter, X1 12MHz

Commit message: BIG UPDATE! omg so big
New boards and other things.. jeesh it sbeen too long since the last update
Parts:
- added U5: SSD1306, afx-01:SSD1306_XL, F.Cu at (137.2, 48.3)
- moved C11 119.3 mm to (109.7, 34.0)
- moved C12 119.3 mm to (122.4, 37.3)
- moved C20 119.3 mm to (104.1, 34.3)
- moved J1 119.3 mm to (116.2, 26.0)
- moved J2 119.3 mm to (92.7, 40.0)
- moved P1 119.3 mm to (136.5, 67.9)
- moved P2 119.3 mm to (146.7, 67.9)
- moved R18 119.3 mm to (123.2, 71.8)
- moved R19 119.3 mm to (116.8, 71.8)
- moved R4 119.3 mm to (108.2, 29.5)
- moved R5 119.3 mm to (122.4, 34.3)
- moved R7 119.3 mm to (104.1, 27.9)
- moved REF** 119.3 mm to (94.6, 27.9)
- moved U1 119.3 mm to (137.2, 27.9)
- moved U4 119.3 mm to (140.3, 48.3)
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Routing:
- net GND: track 608.6 -> 941.3 mm, vias 7 -> 14
- net VCC: track 549.5 -> 748.1 mm, vias 12 -> 18
- net /SwitchMatrix/SDA: track 0.45 -> 151.7 mm, vias 0 -> 4
- net /SwitchMatrix/SCL: track 0.00 -> 149.8 mm, vias 0 -> 2
- net Net-(MCP2-Pad23): track 6.60 -> 133.0 mm, vias 0 -> 1
- net Net-(MCP2-Pad27): track 6.60 -> 126.5 mm, vias 0 -> 1
- net AGND: track 93.3 -> 196.6 mm
- net Net-(ENC1-Pad4): track 0.00 -> 93.8 mm, vias 0 -> 1
- net /SoundBoard/MIDIIN: track 3.30 -> 93.2 mm
- net Net-(MCP1-Pad19): track 6.60 -> 94.5 mm, vias 0 -> 2
- net /SwitchMatrix/ENCB: track 2.71 -> 88.0 mm
- net Net-(MCP1-Pad17): track 6.60 -> 91.3 mm, vias 0 -> 2
- net /SwitchMatrix/ENCA: track 2.71 -> 84.7 mm
- net Net-(C20-Pad1): track 0.00 -> 82.0 mm, vias 0 -> 2
- net Net-(C11-Pad1): track 0.00 -> 77.7 mm, vias 0 -> 2
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Other:
- board size 114.3 x 110.5 mm -> 91.4 x 116.8 mm
