File: sam2695.sch (KiCad schematic (older format))
At the start: 31 parts, among them J1 HeadphoneOut, J2 MicIn, U3 SAM2695, X1 12MHz

Commit message: BIG UPDATE! omg so big
New boards and other things.. jeesh it sbeen too long since the last update
Parts:
- J1, J2: footprint afx-01:Switchcraft_3.5mm_SMD_Stereo -> Zetaohm:Switchcraft_3.5mm_SMD_Stereo
- X1: footprint afx-01:Xtal_3.2mm -> Zetaohm:Xtal_3.2mm
Connections:
- net labels added: +3V3, GNDA
- net labels removed: AGND, GND
- wire segments 133 -> 196
Other:
- moved on the sheet: C10, C11, C12, C13, C14, C15, C16, C17, C18, C19, C20, C21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

Commit message: UPDATEUPDATES!!!
Connections:
- wire segments 196 -> 136
Changed lines of the file:
@@
 $EndComp
 $Comp
-L VCC #PWR016
+L VCC #PWR033
 U 1 1 55727FD6
 P 7650 4400
-F 0 "#PWR016" H 7650 4250 50  0001 C CNN
+F 0 "#PWR033" H 7650 4250 50  0001 C CNN
 F 1 "VCC" H 7650 4550 50  0000 C CNN
 F 2 "" H 7650 4400 60  0000 C CNN
@@
 $EndComp
 $Comp
-L VCC #PWR018
+L VCC #PWR034
 U 1 1 55728291
 P 4250 3200
-F 0 "#PWR018" H 4250 3050 50  0001 C CNN
+F 0 "#PWR034" H 4250 3050 50  0001 C CNN
 F 1 "VCC" H 4250 3350 50  0000 C CNN
 F 2 "" H 4250 3200 60  0000 C CNN
@@
 $EndComp
 $Comp
-L VCC #PWR019
+L VCC #PWR035
 U 1 1 5572872F
 P 8050 3250
-F 0 "#PWR019" H 8050 3100 50  0001 C CNN
+F 0 "#PWR035" H 8050 3100 50  0001 C CNN
 F 1 "VCC" H 8050 3400 50  0000 C CNN
 F 2 "" H 8050 3250 60  0000 C CNN
@@
 NoConn ~ 4650 4000
 $Comp
-L GNDA #PWR?
+L GNDA #PWR036
 U 1 1 561F077A
 P 7150 2400
-F 0 "#PWR?" H 7150 2150 50  0001 C CNN
+F 0 "#PWR036" H 7150 2150 50  0001 C CNN
 F 1 "GNDA" H 7150 2250 50  0000 C CNN
 F 2 "" H 7150 2400 60  0000 C CNN
@@
 $EndComp
 $Comp
-L GNDA #PWR?
+L GNDA #PWR037
 U 1 1 561F07E6
 P 8850 3200
-F 0 "#PWR?" H 8850 2950 50  0001 C CNN
+F 0 "#PWR037" H 8850 2950 50  0001 C CNN
 F 1 "GNDA" H 8850 3050 50  0000 C CNN
 F 2 "" H 8850 3200 60  0000 C CNN
@@
 $EndComp
 $Comp
-L GNDA #PWR?
+L GNDA #PWR038
 U 1 1 561F086A
 P 6250 1900
-F 0 "#PWR?" H 6250 1650 50  0001 C CNN
+F 0 "#PWR038" H 6250 1650 50  0001 C CNN
 F 1 "GNDA" H 6250 1750 50  0000 C CNN
 F 2 "" H 6250 1900 60  0000 C CNN
@@
 $EndComp
 $Comp
-L GNDA #PWR?
+L GNDA #PWR039
 U 1 1 561F08CF
 P 8000 3600
-F 0 "#PWR?" H 8000 3350 50  0001 C CNN
+F 0 "#PWR039" H 8000 3350 50  0001 C CNN
 F 1 "GNDA" H 8000 3450 50  0000 C CNN
 F 2 "" H 8000 3600 60  0000 C CNN
@@
 $EndComp
 $Comp
-L GNDA #PWR?
+L GNDA #PWR040
 U 1 1 561F0AFD
 P 5400 5500
-F 0 "#PWR?" H 5400 5250 50  0001 C CNN
+F 0 "#PWR040" H 5400 5250 50  0001 C CNN
 F 1 "GNDA" H 5400 5350 50  0000 C CNN
 F 2 "" H 5400 5500 60  0000 C CNN
@@
 $EndComp
 $Comp
-L +3V3 #PWR?
+L +3V3 #PWR041
 U 1 1 561F0D6B
 P 4000 3600
-F 0 "#PWR?" H 4000 3450 50  0001 C CNN
+F 0 "#PWR041" H 4000 3450 50  0001 C CNN
 F 1 "+3V3" H 4000 3740 50  0000 C CNN
 F 2 "" H 4000 3600 60  0000 C CNN
@@
 	6300 5000 6200 5000
 Wire Wire Line
-	6300 4700 6300 4850
-Wire Wire Line
-	6300 4850 6300 5000
+	6300 4700 6300 5000
 Wire Wire Line
 	6300 4700 6200 4700
 Connection ~ 6300 4850
 Wire Wire Line
-	5700 4700 5700 4750
-Wire Wire Line
-	5700 4750 5700 4800
+	5700 4700 5700 4800
 Wire Wire Line
 	5700 4700 6050 4700
@@
 	5700 5000 6050 5000
 Wire Wire Line
-	5700 4900 5700 4950
-Wire Wire Line
-	5700 4950 5700 5000
-Wire Wire Line
-	5350 4300 5450 4300
-Wire Wire Line
-	5450 4300 5550 4300
-Wire Wire Line
-	5350 4200 5450 4200
-Wire Wire Line
-	5450 4200 5600 4200
-Wire Wire Line
-	5350 4100 5450 4100
-Wire Wire Line
-	5450 4100 5550 4100
+	5700 4900 5700 5000
+Wire Wire Line
+	5350 4300 5550 4300
+Wire Wire Line
+	5350 4200 5600 4200
+Wire Wire Line
+	5350 4100 5550 4100
 Connection ~ 5450 4200
 Wire Wire Line
-	5350 4000 5450 4000
-Wire Wire Line
-	5450 4000 5550 4000
+	5350 4000 5550 4000
 Connection ~ 5450 4100
 Wire Wire Line
@@
 Connection ~ 5450 4000
 Wire Wire Line
-	5350 3800 5450 3800
-Wire Wire Line
-	5450 3800 6150 3800
+	5350 3800 6150 3800
 Connection ~ 5450 3900
 Connection ~ 5450 3800
 Connection ~ 5450 3700
 Wire Wire Line
-	5350 3700 5450 3700
-Wire Wire Line
-	5450 3700 5600 3700
+	5350 3700 5600 3700
 Wire Wire Line
 	5550 4000 5550 3900
@@
 Connection ~ 5450 4300
 Wire Wire Line
-	6800 3700 6800 3800
-Wire Wire Line
-	6800 3800 6800 3900
-Wire Wire Line
-	6800 3900 6800 4050
-Wire Wire Line
-	6800 4050 6800 4200
-Wire Wire Line
-	6800 4200 6800 4350
-Wire Wire Line
-	7450 5350 7450 4650
-Wire Wire Line
-	7450 4650 7450 4350
+	6800 3700 6800 4350
+Wire Wire Line
+	7450 5350 7450 4350
 Wire Wire Line
 	6800 3800 6300 3800
@@
 Connection ~ 6800 3800
 Wire Wire Line
-	5800 4050 6800 4050
-Wire Wire Line
-	6800 4050 6950 4050
+	5800 4050 6950 4050
 Connection ~ 6800 3900
 Wire Wire Line
@@
 Connection ~ 6800 4050
 Wire Wire Line
-	5800 4350 6800 4350
-Wire Wire Line
-	6800 4350 7450 4350
+	7450 4350 5800 4350
 Connection ~ 6800 4200
 Wire Wire Line
 	4500 5350 4500 5100
 Wire Wire Line
-	4500 5100 4550 5100
-Wire Wire Line
-	4550 5100 4650 5100
+	4500 5100 4650 5100
 Connection ~ 7450 4350
 Wire Wire Line
 	4650 4500 4550 4500
 Wire Wire Line
-	4550 4500 4550 4600
-Wire Wire Line
-	4550 4600 4550 4700
-Wire Wire Line
-	4550 4700 4550 4800
-Wire Wire Line
-	4550 4800 4550 4900
-Wire Wire Line
-	4550 4900 4550 5000
-Wire Wire Line
-	4550 5000 4550 5100
+	4550 4500 4550 5100
 Wire Wire Line
 	4550 4600 4650 4600
@@
 Connection ~ 4550 5000
 Wire Wire Line
-	5350 4450 5450 4450
-Wire Wire Line
-	5450 4450 7650 4450
+	5350 4450 7650 4450
 Wire Wire Line
 	6300 4850 6400 4850
 Wire Wire Line
-	6400 5350 6400 4850
+	6400 4850 6400 5350
 Connection ~ 6400 5350
 Wire Wire Line
 	5350 5100 5400 5100
 Wire Wire Line
-	5400 5100 5400 5350
-Wire Wire Line
-	5400 5350 5400 5500
+	5400 5100 5400 5500
 Connection ~ 5400 5350
 Wire Wire Line
@@
 	4200 3750 4200 3850
 Wire Wire Line
-	3800 3750 4000 3750
-Wire Wire Line
-	4000 3750 4200 3750
+	3800 3750 4200 3750
 Wire Wire Line
 	3800 3750 3800 3850
@@
 	4650 3050 4550 3050
 Wire Wire Line
-	4550 3050 4550 3150
-Wire Wire Line
-	4550 3150 4550 3400
+	4550 3050 4550 3400
 Wire Wire Line
 	4550 3150 4650 3150
 Wire Wire Line
-	3500 3400 4550 3400
-Wire Wire Line
-	4550 3400 4650 3400
+	3500 3400 4650 3400
 Wire Wire Line
 	3500 5350 3500 3400
@@
 	6850 3350 6850 3500
 Wire Wire Line
-	6950 3500 6850 3500
-Wire Wire Line
-	6850 3500 6800 3500
-Wire Wire Line
-	6950 3350 6950 3450
-Wire Wire Line
-	6950 3450 6950 3500
-Wire Wire Line
-	6950 3500 6950 3600
+	6950 3500 6800 3500
+Wire Wire Line
+	6950 3350 6950 3600
 Wire Wire Line
 	6950 3450 7000 3450
@@
 Connection ~ 6950 3450
 Wire Wire Line
-	7200 3450 7750 3450
-Wire Wire Line
-	7750 3450 8000 3450
+	7200 3450 8000 3450
 Wire Wire Line
 	7750 3600 7300 3600
@@
 	6200 3350 6200 3250
 Wire Wire Line
-	6200 3250 6850 3250
-Wire Wire Line
-	6850 3250 7750 3250
-Wire Wire Line
-	5450 3600 5450 3700
-Wire Wire Line
-	5450 3700 5450 3800
-Wire Wire Line
-	5450 3800 5450 3900
-Wire Wire Line
-	5450 3900 5450 4000
-Wire Wire Line
-	5450 4000 5450 4100
-Wire Wire Line
-	5450 4100 5450 4200
-Wire Wire Line
-	5450 4200 5450 4300
-Wire Wire Line
-	5450 4300 5450 4450
+	6200 3250 7750 3250
+Wire Wire Line
+	5450 3600 5450 4450
 Wire Wire Line
 	5450 3600 6100 3600
@@
 	5950 3500 5350 3500
 Wire Wire Line
-	5950 2950 5950 3150
-Wire Wire Line
-	5950 3150 5950 3500
+	5950 2950 5950 3500
 Wire Wire Line
 	5950 3150 6150 3150
@@
 Connection ~ 7750 3250
 Wire Wire Line
-	6850 2950 6850 3150
-Wire Wire Line
-	6850 3150 6850 3250
+	6850 2950 6850 3250
 Connection ~ 6850 3150
 Connection ~ 6850 3250
@@
 	6300 3150 6850 3150
 Wire Wire Line
-	7750 3250 7750 3450
-Wire Wire Line
-	7750 3450 7750 3600
-Wire Wire Line
-	7750 3600 7750 3750
+	7750 3250 7750 3750
 Wire Wire Line
 	5800 3700 6800 3700
@@
 	5400 3000 5350 3000
 Wire Wire Line
-	5850 1650 6250 1650
-Wire Wire Line
-	6250 1650 7650 1650
+	5850 1650 7650 1650
 Wire Wire Line
 	6250 1850 6250 1900
 Wire Wire Line
-	5850 2100 7150 2100
-Wire Wire Line
-	7150 2100 7500 2100
-Wire Wire Line
-	7150 2300 7150 2350
-Wire Wire Line
-	7150 2350 7150 2400
+	5850 2100 7500 2100
+Wire Wire Line
+	7150 2300 7150 2400
 Connection ~ 6250 1650
 Wire Wire Line
@@
 	8850 2950 8950 2950
 Wire Wire Line
-	8850 2750 8850 2800
-Wire Wire Line
-	8850 2800 8850 2850
-Wire Wire Line
-	8850 2850 8850 2950
-Wire Wire Line
-	8850 2950 8850 3100
-Wire Wire Line
-	8850 3100 8850 3200
-Wire Wire Line
-	8300 3100 8500 3100
-Wire Wire Line
-	8500 3100 8850 3100
+	8850 2750 8850 3200
+Wire Wire Line
+	8300 3100 8850 3100
 Connection ~ 8850 3100
 Wire Wire Line
@@
 Connection ~ 8500 3100
 Wire Wire Line
-	7900 2750 8300 2750
-Wire Wire Line
-	8300 2750 8500 2750
+	7900 2750 8500 2750
 Wire Wire Line
 	8500 2750 8500 2900
@@
 	5350 4600 6500 4600
 Wire Wire Line
-	6500 4600 6500 4650
-Wire Wire Line
-	6500 4650 6500 4900
+	6500 4600 6500 4900
 Wire Wire Line
 	6500 4650 6700 4650
@@
 Connection ~ 6500 4650
 Wire Wire Line
-	6850 4650 7100 4650
-Wire Wire Line
-	7100 4650 7450 4650
+	6850 4650 7450 4650
 Connection ~ 7450 4650
 Wire Wire Line
@@
 	4000 4850 4000 5350
 Wire Wire Line
-	3500 5350 4000 5350
-Wire Wire Line
-	4000 5350 4500 5350
-Wire Wire Line
-	4500 5350 5400 5350
-Wire Wire Line
-	5400 5350 6400 5350
-Wire Wire Line
-	6400 5350 7450 5350
+	3500 5350 7450 5350
 Connection ~ 4000 5350
 Connection ~ 6850 3500
@@
 Connection ~ 4000 3750
 Wire Wire Line
-	3800 4150 4000 4150
-Wire Wire Line
-	4000 4150 4200 4150
-Wire Wire Line
-	4000 4150 4000 4250
-Wire Wire Line
-	4000 4250 4000 4700
+	3800 4150 4200 4150
+Wire Wire Line
+	4000 4150 4000 4700
 Connection ~ 4000 4250
 Connection ~ 4000 4150
