File: switchMatrix.sch (KiCad schematic (older format))
At the start: 34 parts

Commit message: BIG UPDATE! omg so big
New boards and other things.. jeesh it sbeen too long since the last update
Parts:
- ENC1: footprint afx-01:AB2_ROTARY_ENCODER_W_SWITCH -> Zetaohm:AB2_ROTARY_ENCODER_W_SWITCH
- S1, S10, S11, S12, S13, S14, S15, S16, S2, S3, S4, S5, S6, S7, S8, S9, SS1, SS2, SS3, SS4, SS5, SS6, SS7, SS8, SS9: footprint afx-01:B3F-1050_6mm_Switch -> Zetaohm:B3F-1050_6mm_Switch
Connections:
- net SCL renamed SCL0
- net SDA renamed SDA0

Commit message: UPDATEUPDATES!!!
Parts:
- removed S16, SS9: DPST_Switch, Zetaohm:B3F-1050_6mm_Switch, symbol DPST_Switch-RESCUE-afx-01
- added C35, C36: .01µf, Capacitors_SMD:C_0805_HandSoldering, symbol Cap
- added ENC1: Encoder_switch, Zetaohm:AB2_ROTARY_ENCODER_W_SWITCH, symbol Encoder_switch
- added J19, J20, J21, J22: Mono_AudioConnector, Zetaohm:THONKICONN, symbol Mono_AudioConnector
- added R47, R48, R49, R50: 10k, Resistors_SMD:R_0805_HandSoldering, symbol Resistor
- added R74, R75, R76, R77: 1k, Resistors_SMD:R_0805_HandSoldering, symbol Resistor
- added S1, SS0: DPST_Switch, Zetaohm:B3F-1050_6mm_Switch, symbol DPST_Switch-RESCUE-afx-01
- renumbered ENC1 to ENC2, S1 to S0
Connections:
- net GND: now also C35.2, C36.2, ENC1.2 (C), ENC1.5 (D), J19.1, J20.1, J21.1, J22.1, S1.3, S1.4, SS0.3, SS0.4
- net VCC: now also R48.2, R49.2
- net S4: now reaches S4.1, S4.2
- net S4: now also MCP1.21 (GPA4); no longer MCP1.1 (GPB4)
- net S0: now reaches MCP1.17 (GPA0), S0.1, S0.2
- net S5: now reaches S5.1, S5.2
- net S5: now also MCP1.22 (GPA5); no longer MCP1.18 (GPA1)
- net S9: now reaches S9.1, S9.2
- net S9: now also MCP1.26 (GPB1); no longer MCP1.19 (GPA2)
- net S8: now reaches S8.1, S8.2
- net S8: now also MCP1.25 (GPB0); no longer MCP1.2 (GPB5)
- net SD: now reaches S13.1, S13.2
- net SD: now also MCP1.2 (GPB5); no longer MCP1.20 (GPA3)
- net S2: now reaches S2.1, S2.2
- net S2: now also MCP1.19 (GPA2); no longer MCP1.21 (GPA4)
- net S6: now reaches S6.1, S6.2
- net S6: now also MCP1.23 (GPA6); no longer MCP1.22 (GPA5)
- net SA: now reaches S10.1, S10.2
- net SA: now also MCP1.27 (GPB2); no longer MCP1.23 (GPA6)
- net SE: now reaches S14.1, S14.2
- net SE: now also MCP1.3 (GPB6); no longer MCP1.24 (GPA7)
- net S3: now reaches S3.1, S3.2
- net S3: now also MCP1.20 (GPA3); no longer MCP1.25 (GPB0)
- net S7: now reaches S7.1, S7.2
- net S7: now also MCP1.24 (GPA7); no longer MCP1.26 (GPB1)
- net SB: now reaches S11.1, S11.2
- net SB: now also MCP1.28 (GPB3); no longer MCP1.27 (GPB2)
- net SF: now reaches S15.1, S15.2
- net SF: now also MCP1.4 (GPB7); no longer MCP1.28 (GPB3)
- net SC: now reaches S12.1, S12.2
- net SC: now also MCP1.1 (GPB4); no longer MCP1.3 (GPB6)
- net ENC2SW: now reaches ENC2.4 (E)
- net ENC2SW: now also MCP2.27 (GPB2); no longer MCP2.1 (GPB4)
- net SS1: now reaches SS1.1, SS1.2
- net SS1: now also MCP2.18 (GPA1); no longer MCP2.17 (GPA0)
- net SS4: now reaches SS4.1, SS4.2
- net SS4: now also MCP2.21 (GPA4); no longer MCP2.18 (GPA1)
- net SS7: now reaches SS7.1, SS7.2
- net SS7: now also MCP2.24 (GPA7); no longer MCP2.19 (GPA2)
- net GATE_OUT2: now reaches MCP2.2 (GPB5)
- net GATE_OUT2: now also R75.2
- net SS3: now reaches MCP2.20 (GPA3)
- net SS3: now also SS3.1, SS3.2
- net SS2: now reaches SS2.1, SS2.2
- net SS2: now also MCP2.19 (GPA2); no longer MCP2.21 (GPA4)
- net SS5: now reaches MCP2.22 (GPA5), SS5.1, SS5.2
- net SS8: now reaches SS8.1, SS8.2
- net SS8: now also MCP2.25 (GPB0); no longer MCP2.23 (GPA6)
- net SS6: now reaches SS6.1, SS6.2
- net SS6: now also MCP2.23 (GPA6); no longer MCP2.26 (GPB1)
- net GATE_OUT3: now reaches MCP2.3 (GPB6)
- net GATE_OUT3: now also R76.2
- net GATE_OUT4: now reaches MCP2.4 (GPB7)
- net GATE_OUT4: now also R77.2
- net ENCA renamed ENC2A
- net ENCB renamed ENC2B
- net SCL0 renamed SCL0_5v
- net SDA0 renamed SDA0_5v
- new net: ENC1.1 (A), R47.1, R48.1
- new net: ENC1.3 (B), R49.1, R50.1
- new net: J19.2, J19.3, R74.1
- new net: J20.2, J20.3, R75.1
- new net: J21.2, J21.3, R76.1
- new net: J22.2, J22.3, R77.1
- new net ENC1A: C35.1, R47.2
- new net ENC1B: C36.1, R50.2
- new net ENC1SW: ENC1.4 (E), MCP2.26 (GPB1)
- new net GATE_OUT1: MCP2.1 (GPB4), R74.2
- new net S1: MCP1.18 (GPA1), S1.1, S1.2
- new net SS0: MCP2.17 (GPA0), SS0.1, SS0.2
- no-connect marks 10 -> 4
Other:
- moved on the sheet: C23, C24, ENC2, MCP1, R12, R13, R14, R15, S0
