File: gateInput.sch (KiCad schematic (older format))
At the start: 9 parts, among them J19 Mono_AudioConnector, J20 Mono_AudioConnector, J21 Mono_AudioConnector, J22 Mono_AudioConnector

Commit message: Updating Schematics
Connections:
- net GATE_OUT1: now also MCP2.21 (GPA4); no longer MCP2.1 (GPB4)
- net GATE_OUT2: now also MCP2.22 (GPA5); no longer MCP2.2 (GPB5)
- net GATE_OUT3: now also MCP2.23 (GPA6); no longer MCP2.3 (GPB6)
- net GATE_OUT4: now also MCP2.24 (GPA7); no longer MCP2.4 (GPB7)
- net ENC1SW: no longer names the net of MCP2.27 (GPB2)
- net ENC2SW: no longer names the net of MCP2.28 (GPB3)
Changed lines of the file:
@@
 NoConn ~ 6700 3400
 NoConn ~ 6700 3500
-Text GLabel 7900 3200 2    39   Output ~ 0
-ENC1SW
-Text GLabel 7900 3300 2    39   Output ~ 0
-ENC2SW
-Text GLabel 7900 3700 2    39   Output ~ 0
+Text GLabel 7900 2700 2    39   Output ~ 0
 GATE_OUT4
-Text GLabel 7900 3600 2    39   Output ~ 0
+Text GLabel 7900 2600 2    39   Output ~ 0
 GATE_OUT3
-Text GLabel 7900 3500 2    39   Output ~ 0
+Text GLabel 7900 2500 2    39   Output ~ 0
 GATE_OUT2
-Text GLabel 7900 3400 2    39   Output ~ 0
+Text GLabel 7900 2400 2    39   Output ~ 0
 GATE_OUT1
 Text GLabel 5750 2200 0    59   Input ~ 0
