File: ADC_Connectors.sch (KiCad schematic (older format))
At the start: 37 parts, among them J11 Mono_AudioConnector, J12 Mono_AudioConnector, J13 Mono_AudioConnector, J14 Mono_AudioConnector, J15 Mono_AudioConnector, J16 Mono_AudioConnector, J17 Mono_AudioConnector, J18 Mono_AudioConnector, Q1 Q_NPN_BCE, Q2 Q_NPN_BCE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

Commit message: Added Touch Capacitive Panel
Parts:
- Q1, Q2, Q3, Q4: value Q_NPN_BCE -> BSS138
Other:
- moved on the sheet: C37, C38, C39, C40, J11, J12, J13, J14, J15, J16, J17, J18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

Commit message: Updating Schematics
Parts:
- added J? (x4): Mono_AudioConnector, Zetaohm:THONKICONN, symbol Mono_AudioConnector
- added MCP?: MCP23017-QFN, Housings_DFN_QFN:QFN-28-1EP_6x6mm_Pitch0.65mm, symbol MCP23017-QFN
- added R? (x4): 1k, Resistors_SMD:R_0805_HandSoldering, symbol Resistor
Connections:
- net GATE_IN1: now also MCP?.17 (GPA0)
- net GATE_IN2: now also MCP?.18 (GPA1)
- net GATE_IN3: now also MCP?.19 (GPA2)
- net GATE_IN4: now also MCP?.20 (GPA3)
- net GND: now also J?.1, J?.1, J?.1, J?.1, MCP?.12 (A1), MCP?.13 (A2), MCP?.6 (VSS)
- new net: J?.2, J?.3, R?.1 (x4)
- new net +5V: MCP?.11 (A0), MCP?.14 (~RESET), MCP?.5 (VDD)
- new net ENC1SW: MCP?.25 (GPB0)
- new net GATE_OUT1: MCP?.21 (GPA4), R?.2
- new net GATE_OUT2: MCP?.22 (GPA5), R?.2
- new net GATE_OUT3: MCP?.23 (GPA6), R?.2
- new net GATE_OUT4: MCP?.24 (GPA7), R?.2
- new net SCL0_5v: MCP?.8 (SCL)
- new net SDA0_5v: MCP?.9 (SDA)
- no-connect marks 0 -> 2
Other:
- moved on the sheet: C37, C38, C39, C40, J11, J12, J13, J14, J15, J16, J17, J18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

Commit message: Updating footprints
Parts:
- added JP6, JP7: JUMPER3, Zetaohm:Jumper_3way, symbol JUMPER3
- C37, C38, C39, C40: footprint Capacitors_SMD:C_0805_HandSoldering -> Capacitors_SMD:C_0603_HandSoldering
- R12, R13, R14, R7: renamed from R?; footprint Resistors_SMD:R_0805_HandSoldering -> Resistors_SMD:R_0603_HandSoldering
- R51, R52, R53, R54, R55, R56, R57, R58, R59, R60, R61, R62, R63, R64, R65, R66, R67, R68, R69, R70: footprint Resistors_SMD:R_0805_HandSoldering -> Resistors_SMD:R_0603_HandSoldering
- gave numbers to parts that had none: 5
Connections:
- net GATE_IN1 renamed MCP_GATE_IN1
- net GATE_IN2 renamed MCP_GATE_IN2
- net GATE_IN3 renamed JUMPER_GATE_IN3
- net JUMPER_GATE_IN3: now also JP6.1, JP6.2; no longer MCP1.19 (GPA2)
- net GATE_IN4 renamed JUMPER_GATE_IN4
- net JUMPER_GATE_IN4: now also JP7.1, JP7.2; no longer MCP1.20 (GPA3)
- new net MCP_GATE_IN3: JP6.3, MCP1.19 (GPA2)
- new net MCP_GATE_IN4: JP7.3, MCP1.20 (GPA3)
Other:
- note added: "GATE 3-4 SELECTOR"
- moved on the sheet: J13, J16, J19, J20, Q2, Q4, R13, R14, R54, R57, R62, R64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

Commit message: Populating pcb file
Parts:
- added J21: Mono_AudioConnector, Zetaohm:THONKICONN, symbol Mono_AudioConnector
- added R89: 1k, Resistors_SMD:R_0603_HandSoldering, symbol Resistor
Connections:
- net ENC1SW: now also MCP1.26 (GPB1); no longer MCP1.25 (GPB0)
- net GND: now also J21.1
- new net: J21.2, J21.3, R89.1
- new net CLOCK_OUT: MCP1.25 (GPB0), R89.2
Changed lines of the file:
@@
 $EndDescr
 $Comp
-L VSS #PWR059
+L VSS #PWR60
 U 1 1 561FE672
 P 1250 1150
-F 0 "#PWR059" H 1250 1000 50  0001 C CNN
+F 0 "#PWR60" H 1250 1000 50  0001 C CNN
 F 1 "VSS" H 1250 1300 50  0000 C CNN
 F 2 "" H 1250 1150 60  0000 C CNN
@@
 $EndComp
 $Comp
-L GND #PWR060
+L GND #PWR62
 U 1 1 561FE686
 P 2050 1850
-F 0 "#PWR060" H 2050 1600 50  0001 C CNN
+F 0 "#PWR62" H 2050 1600 50  0001 C CNN
 F 1 "GND" H 2050 1700 50  0000 C CNN
 F 2 "" H 2050 1850 60  0000 C CNN
@@
 $EndComp
 $Comp
-L +3V3 #PWR061
+L +3V3 #PWR88
 U 1 1 561FE69A
 P 4200 6150
-F 0 "#PWR061" H 4200 6000 50  0001 C CNN
+F 0 "#PWR88" H 4200 6000 50  0001 C CNN
 F 1 "+3V3" H 4200 6290 50  0000 C CNN
 F 2 "" H 4200 6150 60  0000 C CNN
@@
 $EndComp
 $Comp
-L GND #PWR062
+L GND #PWR91
 U 1 1 56204E84
 P 4200 6950
-F 0 "#PWR062" H 4200 6700 50  0001 C CNN
+F 0 "#PWR91" H 4200 6700 50  0001 C CNN
 F 1 "GND" H 4200 6800 50  0000 C CNN
 F 2 "" H 4200 6950 60  0000 C CNN
@@
 $EndComp
 $Comp
-L GND #PWR063
+L GND #PWR61
 U 1 1 562058BD
 P 1400 1850
-F 0 "#PWR063" H 1400 1600 50  0001 C CNN
+F 0 "#PWR61" H 1400 1600 50  0001 C CNN
 F 1 "GND" H 1400 1700 50  0000 C CNN
 F 2 "" H 1400 1850 60  0000 C CNN
@@
 	3100 1650 3450 1650
 $Comp
-L VSS #PWR064
+L VSS #PWR68
 U 1 1 56205D14
 P 1250 2800
-F 0 "#PWR064" H 1250 2650 50  0001 C CNN
+F 0 "#PWR68" H 1250 2650 50  0001 C CNN
 F 1 "VSS" H 1250 2950 50  0000 C CNN
 F 2 "" H 1250 2800 60  0000 C CNN
@@
 $EndComp
 $Comp
-L GND #PWR065
+L GND #PWR72
 U 1 1 56205D1A
 P 2050 3500
-F 0 "#PWR065" H 2050 3250 50  0001 C CNN
+F 0 "#PWR72" H 2050 3250 50  0001 C CNN
 F 1 "GND" H 2050 3350 50  0000 C CNN
 F 2 "" H 2050 3500 60  0000 C CNN
@@
 $EndComp
 $Comp
-L GND #PWR066
+L GND #PWR71
 U 1 1 56205D44
 P 1400 3500
-F 0 "#PWR066" H 1400 3250 50  0001 C CNN
+F 0 "#PWR71" H 1400 3250 50  0001 C CNN
 F 1 "GND" H 1400 3350 50  0000 C CNN
 F 2 "" H 1400 3500 60  0000 C CNN
@@
 	3100 3300 3450 3300
 $Comp
-L VSS #PWR067
+L VSS #PWR76
 U 1 1 56205F0C
 P 1250 4350
-F 0 "#PWR067" H 1250 4200 50  0001 C CNN
+F 0 "#PWR76" H 1250 4200 50  0001 C CNN
 F 1 "VSS" H 1250 4500 50  0000 C CNN
 F 2 "" H 1250 4350 60  0000 C CNN
@@
 $EndComp
 $Comp
-L GND #PWR068
+L GND #PWR81
 U 1 1 56205F12
 P 2050 5050
-F 0 "#PWR068" H 2050 4800 50  0001 C CNN
+F 0 "#PWR81" H 2050 4800 50  0001 C CNN
 F 1 "GND" H 2050 4900 50  0000 C CNN
 F 2 "" H 2050 5050 60  0000 C CNN
@@
 $EndComp
 $Comp
-L GND #PWR069
+L GND #PWR80
 U 1 1 56205F3C
 P 1400 5050
-F 0 "#PWR069" H 1400 4800 50  0001 C CNN
+F 0 "#PWR80" H 1400 4800 50  0001 C CNN
 F 1 "GND" H 1400 4900 50  0000 C CNN
 F 2 "" H 1400 5050 60  0000 C CNN
@@
 	3100 4850 3450 4850
 $Comp
-L VSS #PWR070
+L VSS #PWR87
 U 1 1 56205F58
 P 1250 6000
-F 0 "#PWR070" H 1250 5850 50  0001 C CNN
+F 0 "#PWR87" H 1250 5850 50  0001 C CNN
 F 1 "VSS" H 1250 6150 50  0000 C CNN
 F 2 "" H 1250 6000 60  0000 C CNN
@@
 $EndComp
 $Comp
-L GND #PWR071
+L GND #PWR90
 U 1 1 56205F5E
 P 2050 6700
-F 0 "#PWR071" H 2050 6450 50  0001 C CNN
+F 0 "#PWR90" H 2050 6450 50  0001 C CNN
 F 1 "GND" H 2050 6550 50  0000 C CNN
 F 2 "" H 2050 6700 60  0000 C CNN
@@
 $EndComp
 $Comp
-L GND #PWR072
+L GND #PWR89
 U 1 1 56205F88
 P 1400 6700
-F 0 "#PWR072" H 1400 6450 50  0001 C CNN
+F 0 "#PWR89" H 1400 6450 50  0001 C CNN
 F 1 "GND" H 1400 6550 50  0000 C CNN
 F 2 "" H 1400 6700 60  0000 C CNN
@@
 $EndComp
 $Comp
-L GND #PWR073
+L GND #PWR64
 U 1 1 56206415
 P 8850 2050
-F 0 "#PWR073" H 8850 1800 50  0001 C CNN
+F 0 "#PWR64" H 8850 1800 50  0001 C CNN
 F 1 "GND" H 8850 1900 50  0000 C CNN
 F 2 "" H 8850 2050 60  0000 C CNN
@@
 $EndComp
 $Comp
-L +3V3 #PWR074
+L +3V3 #PWR59
 U 1 1 56206549
 P 8850 1000
-F 0 "#PWR074" H 8850 850 50  0001 C CNN
+F 0 "#PWR59" H 8850 850 50  0001 C CNN
 F 1 "+3V3" H 8850 1140 50  0000 C CNN
 F 2 "" H 8850 1000 60  0000 C CNN
@@
 $EndComp
 $Comp
-L GND #PWR075
+L GND #PWR63
 U 1 1 562068B3
 P 8100 2050
-F 0 "#PWR075" H 8100 1800 50  0001 C CNN
+F 0 "#PWR63" H 8100 1800 50  0001 C CNN
 F 1 "GND" H 8100 1900 50  0000 C CNN
 F 2 "" H 8100 2050 60  0000 C CNN
@@
 $EndComp
 $Comp
-L GND #PWR076
+L GND #PWR78
 U 1 1 5620767E
 P 8450 4700
-F 0 "#PWR076" H 8450 4450 50  0001 C CNN
+F 0 "#PWR78" H 8450 4450 50  0001 C CNN
 F 1 "GND" H 8450 4550 50  0000 C CNN
 F 2 "" H 8450 4700 60  0000 C CNN
@@
 $EndComp
 $Comp
-L +3V3 #PWR077
+L +3V3 #PWR73
 U 1 1 56207690
 P 8450 3650
-F 0 "#PWR077" H 8450 3500 50  0001 C CNN
+F 0 "#PWR73" H 8450 3500 50  0001 C CNN
 F 1 "+3V3" H 8450 3790 50  0000 C CNN
 F 2 "" H 8450 3650 60  0000 C CNN
@@
 $EndComp
 $Comp
-L GND #PWR078
+L GND #PWR77
 U 1 1 5620769F
 P 7700 4700
-F 0 "#PWR078" H 7700 4450 50  0001 C CNN
+F 0 "#PWR77" H 7700 4450 50  0001 C CNN
 F 1 "GND" H 7700 4550 50  0000 C CNN
 F 2 "" H 7700 4700 60  0000 C CNN
@@
 $EndComp
 $Comp
-L GND #PWR079
+L GND #PWR70
 U 1 1 562079A1
 P 10100 3250
-F 0 "#PWR079" H 10100 3000 50  0001 C CNN
+F 0 "#PWR70" H 10100 3000 50  0001 C CNN
 F 1 "GND" H 10100 3100 50  0000 C CNN
 F 2 "" H 10100 3250 60  0000 C CNN
@@
 $EndComp
 $Comp
-L +3V3 #PWR080
+L +3V3 #PWR66
 U 1 1 562079B3
 P 10100 2200
-F 0 "#PWR080" H 10100 2050 50  0001 C CNN
+F 0 "#PWR66" H 10100 2050 50  0001 C CNN
 F 1 "+3V3" H 10100 2340 50  0000 C CNN
 F 2 "" H 10100 2200 60  0000 C CNN
@@
 $EndComp
 $Comp
-L GND #PWR081
+L GND #PWR69
 U 1 1 562079C2
 P 9350 3250
-F 0 "#PWR081" H 9350 3000 50  0001 C CNN
+F 0 "#PWR69" H 9350 3000 50  0001 C CNN
 F 1 "GND" H 9350 3100 50  0000 C CNN
 F 2 "" H 9350 3250 60  0000 C CNN
@@
 $EndComp
 $Comp
-L GND #PWR082
+L GND #PWR86
 U 1 1 562079DA
 P 9950 5750
-F 0 "#PWR082" H 9950 5500 50  0001 C CNN
+F 0 "#PWR86" H 9950 5500 50  0001 C CNN
 F 1 "GND" H 9950 5600 50  0000 C CNN
 F 2 "" H 9950 5750 60  0000 C CNN
@@
 $EndComp
 $Comp
-L +3V3 #PWR083
+L +3V3 #PWR79
 U 1 1 562079EC
 P 9950 4700
-F 0 "#PWR083" H 9950 4550 50  0001 C CNN
+F 0 "#PWR79" H 9950 4550 50  0001 C CNN
 F 1 "+3V3" H 9950 4840 50  0000 C CNN
 F 2 "" H 9950 4700 60  0000 C CNN
@@
 $EndComp
 $Comp
-L GND #PWR084
+L GND #PWR85
 U 1 1 562079FB
 P 9200 5750
-F 0 "#PWR084" H 9200 5500 50  0001 C CNN
+F 0 "#PWR85" H 9200 5500 50  0001 C CNN
 F 1 "GND" H 9200 5600 50  0000 C CNN
 F 2 "" H 9200 5750 60  0000 C CNN
@@
 $EndComp
 $Comp
-L GND-RESCUE-afx-01 #PWR085
+L GND-RESCUE-afx-01 #PWR67
 U 1 1 562998C7
 P 4400 2400
-F 0 "#PWR085" H 4400 2150 50  0001 C CNN
+F 0 "#PWR67" H 4400 2150 50  0001 C CNN
 F 1 "GND" H 4400 2250 50  0000 C CNN
 F 2 "" H 4400 2400 60  0000 C CNN
@@
 NoConn ~ 5550 2950
 NoConn ~ 5550 3050
-Text GLabel 6750 2550 2    39   Output ~ 0
+Text GLabel 6750 2650 2    39   Output ~ 0
 ENC1SW
 Text GLabel 6750 2250 2    39   Output ~ 0
@@
 $EndComp
 $Comp
-L GND-RESCUE-afx-01 #PWR086
+L GND-RESCUE-afx-01 #PWR74
 U 1 1 562998CA
 P 5000 4250
-F 0 "#PWR086" H 5000 4000 50  0001 C CNN
+F 0 "#PWR74" H 5000 4000 50  0001 C CNN
 F 1 "GND" H 5000 4100 50  0000 C CNN
 F 2 "" H 5000 4250 60  0000 C CNN
@@
 $EndComp
 $Comp
-L GND-RESCUE-afx-01 #PWR087
+L GND-RESCUE-afx-01 #PWR75
 U 1 1 562998CD
 P 6500 4250
-F 0 "#PWR087" H 6500 4000 50  0001 C CNN
+F 0 "#PWR75" H 6500 4000 50  0001 C CNN
 F 1 "GND" H 6500 4100 50  0000 C CNN
 F 2 "" H 6500 4250 60  0000 C CNN
@@
 $EndComp
 $Comp
-L GND-RESCUE-afx-01 #PWR088
+L GND-RESCUE-afx-01 #PWR82
 U 1 1 562998D0
 P 5000 5050
-F 0 "#PWR088" H 5000 4800 50  0001 C CNN
+F 0 "#PWR82" H 5000 4800 50  0001 C CNN
 F 1 "GND" H 5000 4900 50  0000 C CNN
 F 2 "" H 5000 5050 60  0000 C CNN
@@
 $EndComp
 $Comp
-L GND-RESCUE-afx-01 #PWR089
+L GND-RESCUE-afx-01 #PWR83
 U 1 1 562998D3
 P 6500 5050
-F 0 "#PWR089" H 6500 4800 50  0001 C CNN
+F 0 "#PWR83" H 6500 4800 50  0001 C CNN
 F 1 "GND" H 6500 4900 50  0000 C CNN
 F 2 "" H 6500 5050 60  0000 C CNN
@@
 $EndComp
 $Comp
-L +5V #PWR090
+L +5V #PWR65
 U 1 1 562998D4
 P 4400 2200
-F 0 "#PWR090" H 4400 2050 50  0001 C CNN
+F 0 "#PWR65" H 4400 2050 50  0001 C CNN
 F 1 "+5V" H 4400 2340 50  0000 C CNN
 F 2 "" H 4400 2200 60  0000 C CNN
@@
 Text GLabel 5750 6750 0    60   Input ~ 0
 MCP_GATE_IN4
+$Comp
+L Mono_AudioConnector J21
+U 1 1 5629D3A1
+P 8000 5500
+F 0 "J21" H 7900 5650 60  0000 C CNN
+F 1 "Mono_AudioConnector" H 8170 5350 60  0001 C CNN
+F 2 "Zetaohm:THONKICONN" H 7700 5650 60  0001 C CNN
+F 3 "" H 7700 5650 60  0000 C CNN
+	1    8000 5500
+	-1   0    0    1
+$EndComp
+Text GLabel 7250 5400 0    39   Output ~ 0
+CLOCK_OUT
+$Comp
+L Resistor R89
+U 1 1 5629D3A8
+P 7550 5400
+F 0 "R89" V 7650 5500 50  0000 C CNN
+F 1 "1k" V 7650 5300 50  0000 C CNN
+F 2 "Resistors_SMD:R_0603_HandSoldering" V 7480 5400 30  0001 C CNN
+F 3 "" H 7550 5400 30  0000 C CNN
+	1    7550 5400
+	0    1    1    0
+$EndComp
+$Comp
+L GND-RESCUE-afx-01 #PWR84
+U 1 1 5629D3AE
+P 7700 5700
+F 0 "#PWR84" H 7700 5450 50  0001 C CNN
+F 1 "GND" H 7700 5550 50  0000 C CNN
+F 2 "" H 7700 5700 60  0000 C CNN
+F 3 "" H 7700 5700 60  0000 C CNN
+	1    7700 5700
+	1    0    0    -1
+$EndComp
+Wire Wire Line
+	7250 5400 7450 5400
+Wire Wire Line
+	7650 5400 7800 5400
+Wire Wire Line
+	7800 5600 7700 5600
+Wire Wire Line
+	7700 5600 7700 5700
+Wire Wire Line
+	7800 5400 7800 5500
+Text GLabel 6750 2550 2    39   Output ~ 0
+CLOCK_OUT
 $EndSCHEMATC
