File: dacConnectors.sch (KiCad schematic (older format))
At the start: 54 parts

Commit message: UPDATEUPDATES!!!
Parts:
- removed U? (x5): OPA4171, symbol OPA4171
- added unit 2 of U6
- added U7: OPA4171, Housings_SSOP:TSSOP-14_4.4x5mm_Pitch0.65mm, symbol OPA4171
- C27, C28, C29, C30, C31, C32, C33, C34: renamed from C?; footprint (none) -> Capacitors_SMD:C_0805_HandSoldering
- R20, R21, R22, R23, R24, R25, R26, R27, R28, R29, R30, R31, R32, R33, R34, R35, R36, R37, R38, R39, R40, R41, R42, R43, R44, R45, R46: renamed from R?; footprint (none) -> Resistors_SMD:R_0805_HandSoldering
- R71: renamed from 10k; value Resistor -> 10k; footprint (none) -> Resistors_SMD:R_0805_HandSoldering
- U6: renamed from U?; footprint (none) -> Housings_SSOP:TSSOP-14_4.4x5mm_Pitch0.65mm
- U8: renamed from U?; footprint (none) -> Housings_SSOP:TSSOP-20_4.4x6.5mm_Pitch0.65mm
- gave numbers to parts that had none: 8
Connections:
- net VREF_OPA: now also U6.5 (+), U7.10 (+), U7.12 (+), U7.3 (+), U7.5 (+)
- net at C29.1, R30.1: now also U6.7
- net at C29.2, R26.1, R28.2: now also U6.6 (-)
- net at C32.2, R33.1, R35.2: now also U7.9 (-)
- net at C32.1, R37.1: now also U7.8
- net at C34.1, R46.1: now also U7.14
- net at C34.2, R42.1, R44.2: now also U7.13 (-)
- net at C28.2, R21.1, R23.2: now also U7.2 (-)
- net at C28.1, R25.1: now also U7.1
- net at C30.1, R31.1: now also U7.7
- net at C30.2, R27.1, R29.2: now also U7.6 (-)

Commit message: Added Touch Capacitive Panel
Parts:
- C27, C28, C29, C30, C31, C32, C33, C34: footprint Capacitors_SMD:C_0805_HandSoldering -> Capacitors_SMD:C_0603_HandSoldering
- R20, R21, R22, R23, R24, R25, R26, R27, R28, R29, R30, R31, R32, R33, R34, R35, R36, R37, R38, R39, R40, R41, R42, R43, R44, R45, R46, R71: footprint Resistors_SMD:R_0805_HandSoldering -> Resistors_SMD:R_0603_HandSoldering
