File: SSD1327.sch (KiCad schematic (older format))
At the start: 12 parts

Commit message: Small updates
Parts:
- added C57: 22pf 16V, Capacitors_SMD:C_0603_HandSoldering, symbol C_Small
- added C58: 4.7ufT/35v, Capacitors_Tantalum_SMD:TantalC_SizeB_EIA-3528_HandSoldering, symbol CP1_Small
- added C60: 4.7uf, Capacitors_SMD:C_0603_HandSoldering, symbol C_Small
- added D3: D_Schottky, Diodes_SMD:SOD-523, symbol D_Schottky
- added L2: 10uH, Capacitors_SMD:C_0805_HandSoldering, symbol INDUCTOR_SMALL
- added R74: 1.27M_1%, Resistors_SMD:R_0603_HandSoldering, symbol Resistor
- added R75: 113k_1%, Resistors_SMD:R_0603_HandSoldering, symbol Resistor
- C53, C54: renamed from C?; footprint (none) -> Capacitors_Tantalum_SMD:TantalC_SizeB_EIA-3528_HandSoldering
- C55, C56: renamed from C?; footprint (none) -> Capacitors_SMD:C_0603_HandSoldering
- C59: renamed from C?; value C_Small -> 100nf; footprint (none) -> Capacitors_SMD:C_0603_HandSoldering
- R48, R49, R50: renamed from R?; footprint (none) -> Resistors_SMD:R_0603_HandSoldering
- U15: renamed from U?; footprint (none) -> Zetaohm:SSD1327_HOT_BAR
- U16: renamed from U?; footprint (none) -> Zetaohm:VSON-8
- gave numbers to parts that had none: 2
Connections:
- net GND: now also C59.2, U16.6 (GND), U16.7 (PGND), C58.2, C60.2, R75.1
- net at U16.1 (L): now also C60.1, L2.1
- net +5V: now reaches U16.2 (VIN)
- net +5V: now also C59.1
- net at U16.4 (FB): now also C57.2, R74.1, R75.2
- net at U16.8 (SW): now also D3.2 (A), L2.2
- net +12V renamed +3V3
- net +3V3: no longer C53.1, U15.2 (VCC), U15.24 (VCC)
- new net +15V: C53.1, C57.1, C58.1, D3.1 (K), R74.2, U15.2 (VCC), U15.24 (VCC)
Other:
- moved on the sheet: C59, U16
